File: Prototype Schematics/inventeam_proto_schematics/Thermistor Logic Schematic.kicad_sch (KiCad schematic)
At the start: 43 parts, among them J1 Conn_02x20_Top_Bottom, J2 Conn_01x03, J3 Screw_Terminal_01x02, U1 MCP23S17_SP, U2 TMUX1208PW, U3 MCP23S17_SP, U4 TMUX1208PW, U5 MCP1525-TO, U6 OPA2333xxD

Commit message: v16 minor 1
Parts:
- renumbered A1 to A2001, BT1 to BT2001, C1 to C2001, C23 to C2002, C2 to C2003, C3 to C2004, C24 to C2005, C4 to C2006, C5 to C2007, C6 to C2008, C7 to C2009, C8 to C2010, C9 to C2011, C10 to C2012, C11 to C2013, F1 to F2001, J1 to J2001, J2 to J2002, J3 to J2003, R1 to R2001, R2 to R2002, R341 to R2003, R3 to R2004, R4 to R2005, R342 to R2006, R5 to R2007, R6 to R2008, R7 to R2009, R8 to R2010, R9 to R2011, R10 to R2012, R11 to R2013, R343 to R2014, R12 to R2015, R344 to R2016, R13 to R2017, R14 to R2018, U1 to U2001, U2 to U2002, U3 to U2003, U4 to U2004, U5 to U2005, U6 to U2006
Other:
- title: Main -> Thermistor Logic Schematic
