File: Prototype Schematics/inventeam_proto_schematics/FSR Matrix Schematic.kicad_sch (KiCad schematic)
At the start: 312 parts

Commit message: v16 minor 1
Parts:
- renumbered R15 to R4001, R16 to R4002, R17 to R4003, R18 to R4004, R19 to R4005, R20 to R4006, R21 to R4007, R22 to R4008, R23 to R4009, R24 to R4010, R25 to R4011, R26 to R4012, R27 to R4013, R28 to R4014, R29 to R4015, R30 to R4016, R31 to R4017, R32 to R4018, R33 to R4019, R34 to R4020, R35 to R4021, R36 to R4022, R37 to R4023, R38 to R4024, R39 to R4025, R40 to R4026, R41 to R4027, R42 to R4028, R43 to R4029, R44 to R4030, R45 to R4031, R46 to R4032, R47 to R4033, R48 to R4034, R49 to R4035, R50 to R4036, R51 to R4037, R52 to R4038, R53 to R4039, R54 to R4040, R55 to R4041, R56 to R4042, R57 to R4043, R58 to R4044, R59 to R4045, R60 to R4046, R61 to R4047, R62 to R4048, R63 to R4049, R64 to R4050, R65 to R4051, R66 to R4052, R67 to R4053, R68 to R4054, R69 to R4055, R70 to R4056, R71 to R4057, R72 to R4058, R73 to R4059, R74 to R4060, R75 to R4061, R76 to R4062, R77 to R4063, R78 to R4064, R79 to R4065, R80 to R4066, R81 to R4067, R82 to R4068, R83 to R4069, R84 to R4070, R85 to R4071, R86 to R4072, R87 to R4073, R88 to R4074, R89 to R4075, R90 to R4076, R91 to R4077, R92 to R4078, R93 to R4079, R94 to R4080, R95 to R4081, R96 to R4082, R97 to R4083, R98 to R4084, R99 to R4085, R100 to R4086, R101 to R4087, R102 to R4088, R103 to R4089, R104 to R4090, R105 to R4091, R106 to R4092, R107 to R4093, R108 to R4094, R109 to R4095, R110 to R4096, R111 to R4097, R112 to R4098, R113 to R4099, R114 to R4100, R115 to R4101, R116 to R4102, R117 to R4103, R118 to R4104, R119 to R4105, R120 to R4106, R121 to R4107, R122 to R4108, R123 to R4109, R124 to R4110, R125 to R4111, R126 to R4112, R127 to R4113, R128 to R4114, R129 to R4115, R130 to R4116, R131 to R4117, R132 to R4118, R133 to R4119, R134 to R4120, R135 to R4121, R136 to R4122, R137 to R4123, R138 to R4124, R139 to R4125, R140 to R4126, R141 to R4127, R142 to R4128, R143 to R4129, R144 to R4130, R145 to R4131, R146 to R4132, R147 to R4133, R148 to R4134, R149 to R4135, R150 to R4136, R151 to R4137, R152 to R4138, R153 to R4139, R154 to R4140, R155 to R4141, R156 to R4142, R157 to R4143, R158 to R4144, R159 to R4145, R160 to R4146, R161 to R4147, R162 to R4148, R163 to R4149, R164 to R4150, R165 to R4151, R166 to R4152, R167 to R4153, R168 to R4154, R169 to R4155, R170 to R4156, R171 to R4157, R172 to R4158, R173 to R4159, R174 to R4160, R175 to R4161, R176 to R4162, R177 to R4163, R178 to R4164, R179 to R4165, R180 to R4166, R181 to R4167, R182 to R4168, R183 to R4169, R184 to R4170, R185 to R4171, R186 to R4172, R187 to R4173, R188 to R4174, R189 to R4175, R190 to R4176, R191 to R4177, R192 to R4178, R193 to R4179, R194 to R4180, R195 to R4181, R196 to R4182, R197 to R4183, R198 to R4184, R199 to R4185, R200 to R4186, R201 to R4187, R202 to R4188, R203 to R4189, R204 to R4190, R205 to R4191, R206 to R4192, R207 to R4193, R208 to R4194, R209 to R4195, R210 to R4196, R211 to R4197, R212 to R4198, R213 to R4199, R214 to R4200, R215 to R4201, R216 to R4202, R217 to R4203, R218 to R4204, R219 to R4205, R220 to R4206, R221 to R4207, R222 to R4208, R223 to R4209, R224 to R4210, R225 to R4211, R226 to R4212, R227 to R4213, R228 to R4214, R229 to R4215, R230 to R4216, R231 to R4217, R232 to R4218, R233 to R4219, R234 to R4220, R235 to R4221, R236 to R4222, R237 to R4223, R238 to R4224, R239 to R4225, R240 to R4226, R241 to R4227, R242 to R4228, R243 to R4229, R244 to R4230, R245 to R4231, R246 to R4232, R247 to R4233, R248 to R4234, R249 to R4235, R250 to R4236, R251 to R4237, R252 to R4238, R253 to R4239, R254 to R4240, R255 to R4241, R256 to R4242, R257 to R4243, R258 to R4244, R259 to R4245, R260 to R4246, R261 to R4247, R262 to R4248, R263 to R4249, R264 to R4250, R265 to R4251, R266 to R4252, R267 to R4253, R268 to R4254, R269 to R4255, R270 to R4256, R271 to R4257, R272 to R4258, R273 to R4259, R274 to R4260, R275 to R4261, R276 to R4262, R277 to R4263, R278 to R4264, R279 to R4265, R280 to R4266, R281 to R4267, R282 to R4268, R283 to R4269, R284 to R4270, R285 to R4271, R286 to R4272, R287 to R4273, R288 to R4274, R289 to R4275, R290 to R4276, R291 to R4277, R292 to R4278, R293 to R4279, R294 to R4280, R295 to R4281, R296 to R4282, R297 to R4283, R298 to R4284, R299 to R4285, R300 to R4286, R301 to R4287, R302 to R4288, R303 to R4289, R304 to R4290, R305 to R4291, R306 to R4292, R307 to R4293, R308 to R4294, R309 to R4295, R310 to R4296, R311 to R4297, R312 to R4298, R313 to R4299, R314 to R4300, R315 to R4301, R316 to R4302, R317 to R4303, R318 to R4304, R319 to R4305, R320 to R4306, R321 to R4307, R322 to R4308, R323 to R4309, R324 to R4310, R325 to R4311, R326 to R4312
Other:
- title: (none) -> FSR Matrix Schematic

Commit message: V17
Parts:
- renumbered R4001 to R5001, R4002 to R5002, R4003 to R5003, R4004 to R5004, R4005 to R5005, R4006 to R5006, R4007 to R5007, R4008 to R5008, R4009 to R5009, R4010 to R5010, R4011 to R5011, R4012 to R5012, R4013 to R5013, R4014 to R5014, R4015 to R5015, R4016 to R5016, R4017 to R5017, R4018 to R5018, R4019 to R5019, R4020 to R5020, R4021 to R5021, R4022 to R5022, R4023 to R5023, R4024 to R5024, R4025 to R5025, R4026 to R5026, R4027 to R5027, R4028 to R5028, R4029 to R5029, R4030 to R5030, R4031 to R5031, R4032 to R5032, R4033 to R5033, R4034 to R5034, R4035 to R5035, R4036 to R5036, R4037 to R5037, R4038 to R5038, R4039 to R5039, R4040 to R5040, R4041 to R5041, R4042 to R5042, R4043 to R5043, R4044 to R5044, R4045 to R5045, R4046 to R5046, R4047 to R5047, R4048 to R5048, R4049 to R5049, R4050 to R5050, R4051 to R5051, R4052 to R5052, R4053 to R5053, R4054 to R5054, R4055 to R5055, R4056 to R5056, R4057 to R5057, R4058 to R5058, R4059 to R5059, R4060 to R5060, R4061 to R5061, R4062 to R5062, R4063 to R5063, R4064 to R5064, R4065 to R5065, R4066 to R5066, R4067 to R5067, R4068 to R5068, R4069 to R5069, R4070 to R5070, R4071 to R5071, R4072 to R5072, R4073 to R5073, R4074 to R5074, R4075 to R5075, R4076 to R5076, R4077 to R5077, R4078 to R5078, R4079 to R5079, R4080 to R5080, R4081 to R5081, R4082 to R5082, R4083 to R5083, R4084 to R5084, R4085 to R5085, R4086 to R5086, R4087 to R5087, R4088 to R5088, R4089 to R5089, R4090 to R5090, R4091 to R5091, R4092 to R5092, R4093 to R5093, R4094 to R5094, R4095 to R5095, R4096 to R5096, R4097 to R5097, R4098 to R5098, R4099 to R5099, R4100 to R5100, R4101 to R5101, R4102 to R5102, R4103 to R5103, R4104 to R5104, R4105 to R5105, R4106 to R5106, R4107 to R5107, R4108 to R5108, R4109 to R5109, R4110 to R5110, R4111 to R5111, R4112 to R5112, R4113 to R5113, R4114 to R5114, R4115 to R5115, R4116 to R5116, R4117 to R5117, R4118 to R5118, R4119 to R5119, R4120 to R5120, R4121 to R5121, R4122 to R5122, R4123 to R5123, R4124 to R5124, R4125 to R5125, R4126 to R5126, R4127 to R5127, R4128 to R5128, R4129 to R5129, R4130 to R5130, R4131 to R5131, R4132 to R5132, R4133 to R5133, R4134 to R5134, R4135 to R5135, R4136 to R5136, R4137 to R5137, R4138 to R5138, R4139 to R5139, R4140 to R5140, R4141 to R5141, R4142 to R5142, R4143 to R5143, R4144 to R5144, R4145 to R5145, R4146 to R5146, R4147 to R5147, R4148 to R5148, R4149 to R5149, R4150 to R5150, R4151 to R5151, R4152 to R5152, R4153 to R5153, R4154 to R5154, R4155 to R5155, R4156 to R5156, R4157 to R5157, R4158 to R5158, R4159 to R5159, R4160 to R5160, R4161 to R5161, R4162 to R5162, R4163 to R5163, R4164 to R5164, R4165 to R5165, R4166 to R5166, R4167 to R5167, R4168 to R5168, R4169 to R5169, R4170 to R5170, R4171 to R5171, R4172 to R5172, R4173 to R5173, R4174 to R5174, R4175 to R5175, R4176 to R5176, R4177 to R5177, R4178 to R5178, R4179 to R5179, R4180 to R5180, R4181 to R5181, R4182 to R5182, R4183 to R5183, R4184 to R5184, R4185 to R5185, R4186 to R5186, R4187 to R5187, R4188 to R5188, R4189 to R5189, R4190 to R5190, R4191 to R5191, R4192 to R5192, R4193 to R5193, R4194 to R5194, R4195 to R5195, R4196 to R5196, R4197 to R5197, R4198 to R5198, R4199 to R5199, R4200 to R5200, R4201 to R5201, R4202 to R5202, R4203 to R5203, R4204 to R5204, R4205 to R5205, R4206 to R5206, R4207 to R5207, R4208 to R5208, R4209 to R5209, R4210 to R5210, R4211 to R5211, R4212 to R5212, R4213 to R5213, R4214 to R5214, R4215 to R5215, R4216 to R5216, R4217 to R5217, R4218 to R5218, R4219 to R5219, R4220 to R5220, R4221 to R5221, R4222 to R5222, R4223 to R5223, R4224 to R5224, R4225 to R5225, R4226 to R5226, R4227 to R5227, R4228 to R5228, R4229 to R5229, R4230 to R5230, R4231 to R5231, R4232 to R5232, R4233 to R5233, R4234 to R5234, R4235 to R5235, R4236 to R5236, R4237 to R5237, R4238 to R5238, R4239 to R5239, R4240 to R5240, R4241 to R5241, R4242 to R5242, R4243 to R5243, R4244 to R5244, R4245 to R5245, R4246 to R5246, R4247 to R5247, R4248 to R5248, R4249 to R5249, R4250 to R5250, R4251 to R5251, R4252 to R5252, R4253 to R5253, R4254 to R5254, R4255 to R5255, R4256 to R5256, R4257 to R5257, R4258 to R5258, R4259 to R5259, R4260 to R5260, R4261 to R5261, R4262 to R5262, R4263 to R5263, R4264 to R5264, R4265 to R5265, R4266 to R5266, R4267 to R5267, R4268 to R5268, R4269 to R5269, R4270 to R5270, R4271 to R5271, R4272 to R5272, R4273 to R5273, R4274 to R5274, R4275 to R5275, R4276 to R5276, R4277 to R5277, R4278 to R5278, R4279 to R5279, R4280 to R5280, R4281 to R5281, R4282 to R5282, R4283 to R5283, R4284 to R5284, R4285 to R5285, R4286 to R5286, R4287 to R5287, R4288 to R5288, R4289 to R5289, R4290 to R5290, R4291 to R5291, R4292 to R5292, R4293 to R5293, R4294 to R5294, R4295 to R5295, R4296 to R5296, R4297 to R5297, R4298 to R5298, R4299 to R5299, R4300 to R5300, R4301 to R5301, R4302 to R5302, R4303 to R5303, R4304 to R5304, R4305 to R5305, R4306 to R5306, R4307 to R5307, R4308 to R5308, R4309 to R5309, R4310 to R5310, R4311 to R5311, R4312 to R5312
