File: Prototype Schematics/inventeam_proto_schematics/Thermistor Matrix Schematic.kicad_sch (KiCad schematic)
At the start: 312 parts

Commit message: v16 minor 1
Parts:
- renumbered TH1 to TH3001, TH2 to TH3002, TH3 to TH3003, TH4 to TH3004, TH5 to TH3005, TH6 to TH3006, TH7 to TH3007, TH8 to TH3008, TH9 to TH3009, TH10 to TH3010, TH11 to TH3011, TH12 to TH3012, TH13 to TH3013, TH14 to TH3014, TH15 to TH3015, TH16 to TH3016, TH17 to TH3017, TH18 to TH3018, TH19 to TH3019, TH20 to TH3020, TH21 to TH3021, TH22 to TH3022, TH23 to TH3023, TH24 to TH3024, TH25 to TH3025, TH26 to TH3026, TH27 to TH3027, TH28 to TH3028, TH29 to TH3029, TH30 to TH3030, TH31 to TH3031, TH32 to TH3032, TH33 to TH3033, TH34 to TH3034, TH35 to TH3035, TH36 to TH3036, TH37 to TH3037, TH38 to TH3038, TH39 to TH3039, TH40 to TH3040, TH41 to TH3041, TH42 to TH3042, TH43 to TH3043, TH44 to TH3044, TH45 to TH3045, TH46 to TH3046, TH47 to TH3047, TH48 to TH3048, TH49 to TH3049, TH50 to TH3050, TH51 to TH3051, TH52 to TH3052, TH53 to TH3053, TH54 to TH3054, TH55 to TH3055, TH56 to TH3056, TH57 to TH3057, TH58 to TH3058, TH59 to TH3059, TH60 to TH3060, TH61 to TH3061, TH62 to TH3062, TH63 to TH3063, TH64 to TH3064, TH65 to TH3065, TH66 to TH3066, TH67 to TH3067, TH68 to TH3068, TH69 to TH3069, TH70 to TH3070, TH71 to TH3071, TH72 to TH3072, TH73 to TH3073, TH74 to TH3074, TH75 to TH3075, TH76 to TH3076, TH77 to TH3077, TH78 to TH3078, TH79 to TH3079, TH80 to TH3080, TH81 to TH3081, TH82 to TH3082, TH83 to TH3083, TH84 to TH3084, TH85 to TH3085, TH86 to TH3086, TH87 to TH3087, TH88 to TH3088, TH89 to TH3089, TH90 to TH3090, TH91 to TH3091, TH92 to TH3092, TH93 to TH3093, TH94 to TH3094, TH95 to TH3095, TH96 to TH3096, TH97 to TH3097, TH98 to TH3098, TH99 to TH3099, TH100 to TH3100, TH101 to TH3101, TH102 to TH3102, TH103 to TH3103, TH104 to TH3104, TH105 to TH3105, TH106 to TH3106, TH107 to TH3107, TH108 to TH3108, TH109 to TH3109, TH110 to TH3110, TH111 to TH3111, TH112 to TH3112, TH113 to TH3113, TH114 to TH3114, TH115 to TH3115, TH116 to TH3116, TH117 to TH3117, TH118 to TH3118, TH119 to TH3119, TH120 to TH3120, TH121 to TH3121, TH122 to TH3122, TH123 to TH3123, TH124 to TH3124, TH125 to TH3125, TH126 to TH3126, TH127 to TH3127, TH128 to TH3128, TH129 to TH3129, TH130 to TH3130, TH131 to TH3131, TH132 to TH3132, TH133 to TH3133, TH134 to TH3134, TH135 to TH3135, TH136 to TH3136, TH137 to TH3137, TH138 to TH3138, TH139 to TH3139, TH140 to TH3140, TH141 to TH3141, TH142 to TH3142, TH143 to TH3143, TH144 to TH3144, TH145 to TH3145, TH146 to TH3146, TH147 to TH3147, TH148 to TH3148, TH149 to TH3149, TH150 to TH3150, TH151 to TH3151, TH152 to TH3152, TH153 to TH3153, TH154 to TH3154, TH155 to TH3155, TH156 to TH3156, TH157 to TH3157, TH158 to TH3158, TH159 to TH3159, TH160 to TH3160, TH161 to TH3161, TH162 to TH3162, TH163 to TH3163, TH164 to TH3164, TH165 to TH3165, TH166 to TH3166, TH167 to TH3167, TH168 to TH3168, TH169 to TH3169, TH170 to TH3170, TH171 to TH3171, TH172 to TH3172, TH173 to TH3173, TH174 to TH3174, TH175 to TH3175, TH176 to TH3176, TH177 to TH3177, TH178 to TH3178, TH179 to TH3179, TH180 to TH3180, TH181 to TH3181, TH182 to TH3182, TH183 to TH3183, TH184 to TH3184, TH185 to TH3185, TH186 to TH3186, TH187 to TH3187, TH188 to TH3188, TH189 to TH3189, TH190 to TH3190, TH191 to TH3191, TH192 to TH3192, TH193 to TH3193, TH194 to TH3194, TH195 to TH3195, TH196 to TH3196, TH197 to TH3197, TH198 to TH3198, TH199 to TH3199, TH200 to TH3200, TH201 to TH3201, TH202 to TH3202, TH203 to TH3203, TH204 to TH3204, TH205 to TH3205, TH206 to TH3206, TH207 to TH3207, TH208 to TH3208, TH209 to TH3209, TH210 to TH3210, TH211 to TH3211, TH212 to TH3212, TH213 to TH3213, TH214 to TH3214, TH215 to TH3215, TH216 to TH3216, TH217 to TH3217, TH218 to TH3218, TH219 to TH3219, TH220 to TH3220, TH221 to TH3221, TH222 to TH3222, TH223 to TH3223, TH224 to TH3224, TH225 to TH3225, TH226 to TH3226, TH227 to TH3227, TH228 to TH3228, TH229 to TH3229, TH230 to TH3230, TH231 to TH3231, TH232 to TH3232, TH233 to TH3233, TH234 to TH3234, TH235 to TH3235, TH236 to TH3236, TH237 to TH3237, TH238 to TH3238, TH239 to TH3239, TH240 to TH3240, TH241 to TH3241, TH242 to TH3242, TH243 to TH3243, TH244 to TH3244, TH245 to TH3245, TH246 to TH3246, TH247 to TH3247, TH248 to TH3248, TH249 to TH3249, TH250 to TH3250, TH251 to TH3251, TH252 to TH3252, TH253 to TH3253, TH254 to TH3254, TH255 to TH3255, TH256 to TH3256, TH257 to TH3257, TH258 to TH3258, TH259 to TH3259, TH260 to TH3260, TH261 to TH3261, TH262 to TH3262, TH263 to TH3263, TH264 to TH3264, TH265 to TH3265, TH266 to TH3266, TH267 to TH3267, TH268 to TH3268, TH269 to TH3269, TH270 to TH3270, TH271 to TH3271, TH272 to TH3272, TH273 to TH3273, TH274 to TH3274, TH275 to TH3275, TH276 to TH3276, TH277 to TH3277, TH278 to TH3278, TH279 to TH3279, TH280 to TH3280, TH281 to TH3281, TH282 to TH3282, TH283 to TH3283, TH284 to TH3284, TH285 to TH3285, TH286 to TH3286, TH287 to TH3287, TH288 to TH3288, TH289 to TH3289, TH290 to TH3290, TH291 to TH3291, TH292 to TH3292, TH293 to TH3293, TH294 to TH3294, TH295 to TH3295, TH296 to TH3296, TH297 to TH3297, TH298 to TH3298, TH299 to TH3299, TH300 to TH3300, TH301 to TH3301, TH302 to TH3302, TH303 to TH3303, TH304 to TH3304, TH305 to TH3305, TH306 to TH3306, TH307 to TH3307, TH308 to TH3308, TH309 to TH3309, TH310 to TH3310, TH311 to TH3311, TH312 to TH3312
Other:
- title: Thermistor Matrix -> Thermistor Matrix Schematic

Commit message: V17
Parts:
- renumbered TH3001 to TH4001, TH3002 to TH4002, TH3003 to TH4003, TH3004 to TH4004, TH3005 to TH4005, TH3006 to TH4006, TH3007 to TH4007, TH3008 to TH4008, TH3009 to TH4009, TH3010 to TH4010, TH3011 to TH4011, TH3012 to TH4012, TH3013 to TH4013, TH3014 to TH4014, TH3015 to TH4015, TH3016 to TH4016, TH3017 to TH4017, TH3018 to TH4018, TH3019 to TH4019, TH3020 to TH4020, TH3021 to TH4021, TH3022 to TH4022, TH3023 to TH4023, TH3024 to TH4024, TH3025 to TH4025, TH3026 to TH4026, TH3027 to TH4027, TH3028 to TH4028, TH3029 to TH4029, TH3030 to TH4030, TH3031 to TH4031, TH3032 to TH4032, TH3033 to TH4033, TH3034 to TH4034, TH3035 to TH4035, TH3036 to TH4036, TH3037 to TH4037, TH3038 to TH4038, TH3039 to TH4039, TH3040 to TH4040, TH3041 to TH4041, TH3042 to TH4042, TH3043 to TH4043, TH3044 to TH4044, TH3045 to TH4045, TH3046 to TH4046, TH3047 to TH4047, TH3048 to TH4048, TH3049 to TH4049, TH3050 to TH4050, TH3051 to TH4051, TH3052 to TH4052, TH3053 to TH4053, TH3054 to TH4054, TH3055 to TH4055, TH3056 to TH4056, TH3057 to TH4057, TH3058 to TH4058, TH3059 to TH4059, TH3060 to TH4060, TH3061 to TH4061, TH3062 to TH4062, TH3063 to TH4063, TH3064 to TH4064, TH3065 to TH4065, TH3066 to TH4066, TH3067 to TH4067, TH3068 to TH4068, TH3069 to TH4069, TH3070 to TH4070, TH3071 to TH4071, TH3072 to TH4072, TH3073 to TH4073, TH3074 to TH4074, TH3075 to TH4075, TH3076 to TH4076, TH3077 to TH4077, TH3078 to TH4078, TH3079 to TH4079, TH3080 to TH4080, TH3081 to TH4081, TH3082 to TH4082, TH3083 to TH4083, TH3084 to TH4084, TH3085 to TH4085, TH3086 to TH4086, TH3087 to TH4087, TH3088 to TH4088, TH3089 to TH4089, TH3090 to TH4090, TH3091 to TH4091, TH3092 to TH4092, TH3093 to TH4093, TH3094 to TH4094, TH3095 to TH4095, TH3096 to TH4096, TH3097 to TH4097, TH3098 to TH4098, TH3099 to TH4099, TH3100 to TH4100, TH3101 to TH4101, TH3102 to TH4102, TH3103 to TH4103, TH3104 to TH4104, TH3105 to TH4105, TH3106 to TH4106, TH3107 to TH4107, TH3108 to TH4108, TH3109 to TH4109, TH3110 to TH4110, TH3111 to TH4111, TH3112 to TH4112, TH3113 to TH4113, TH3114 to TH4114, TH3115 to TH4115, TH3116 to TH4116, TH3117 to TH4117, TH3118 to TH4118, TH3119 to TH4119, TH3120 to TH4120, TH3121 to TH4121, TH3122 to TH4122, TH3123 to TH4123, TH3124 to TH4124, TH3125 to TH4125, TH3126 to TH4126, TH3127 to TH4127, TH3128 to TH4128, TH3129 to TH4129, TH3130 to TH4130, TH3131 to TH4131, TH3132 to TH4132, TH3133 to TH4133, TH3134 to TH4134, TH3135 to TH4135, TH3136 to TH4136, TH3137 to TH4137, TH3138 to TH4138, TH3139 to TH4139, TH3140 to TH4140, TH3141 to TH4141, TH3142 to TH4142, TH3143 to TH4143, TH3144 to TH4144, TH3145 to TH4145, TH3146 to TH4146, TH3147 to TH4147, TH3148 to TH4148, TH3149 to TH4149, TH3150 to TH4150, TH3151 to TH4151, TH3152 to TH4152, TH3153 to TH4153, TH3154 to TH4154, TH3155 to TH4155, TH3156 to TH4156, TH3157 to TH4157, TH3158 to TH4158, TH3159 to TH4159, TH3160 to TH4160, TH3161 to TH4161, TH3162 to TH4162, TH3163 to TH4163, TH3164 to TH4164, TH3165 to TH4165, TH3166 to TH4166, TH3167 to TH4167, TH3168 to TH4168, TH3169 to TH4169, TH3170 to TH4170, TH3171 to TH4171, TH3172 to TH4172, TH3173 to TH4173, TH3174 to TH4174, TH3175 to TH4175, TH3176 to TH4176, TH3177 to TH4177, TH3178 to TH4178, TH3179 to TH4179, TH3180 to TH4180, TH3181 to TH4181, TH3182 to TH4182, TH3183 to TH4183, TH3184 to TH4184, TH3185 to TH4185, TH3186 to TH4186, TH3187 to TH4187, TH3188 to TH4188, TH3189 to TH4189, TH3190 to TH4190, TH3191 to TH4191, TH3192 to TH4192, TH3193 to TH4193, TH3194 to TH4194, TH3195 to TH4195, TH3196 to TH4196, TH3197 to TH4197, TH3198 to TH4198, TH3199 to TH4199, TH3200 to TH4200, TH3201 to TH4201, TH3202 to TH4202, TH3203 to TH4203, TH3204 to TH4204, TH3205 to TH4205, TH3206 to TH4206, TH3207 to TH4207, TH3208 to TH4208, TH3209 to TH4209, TH3210 to TH4210, TH3211 to TH4211, TH3212 to TH4212, TH3213 to TH4213, TH3214 to TH4214, TH3215 to TH4215, TH3216 to TH4216, TH3217 to TH4217, TH3218 to TH4218, TH3219 to TH4219, TH3220 to TH4220, TH3221 to TH4221, TH3222 to TH4222, TH3223 to TH4223, TH3224 to TH4224, TH3225 to TH4225, TH3226 to TH4226, TH3227 to TH4227, TH3228 to TH4228, TH3229 to TH4229, TH3230 to TH4230, TH3231 to TH4231, TH3232 to TH4232, TH3233 to TH4233, TH3234 to TH4234, TH3235 to TH4235, TH3236 to TH4236, TH3237 to TH4237, TH3238 to TH4238, TH3239 to TH4239, TH3240 to TH4240, TH3241 to TH4241, TH3242 to TH4242, TH3243 to TH4243, TH3244 to TH4244, TH3245 to TH4245, TH3246 to TH4246, TH3247 to TH4247, TH3248 to TH4248, TH3249 to TH4249, TH3250 to TH4250, TH3251 to TH4251, TH3252 to TH4252, TH3253 to TH4253, TH3254 to TH4254, TH3255 to TH4255, TH3256 to TH4256, TH3257 to TH4257, TH3258 to TH4258, TH3259 to TH4259, TH3260 to TH4260, TH3261 to TH4261, TH3262 to TH4262, TH3263 to TH4263, TH3264 to TH4264, TH3265 to TH4265, TH3266 to TH4266, TH3267 to TH4267, TH3268 to TH4268, TH3269 to TH4269, TH3270 to TH4270, TH3271 to TH4271, TH3272 to TH4272, TH3273 to TH4273, TH3274 to TH4274, TH3275 to TH4275, TH3276 to TH4276, TH3277 to TH4277, TH3278 to TH4278, TH3279 to TH4279, TH3280 to TH4280, TH3281 to TH4281, TH3282 to TH4282, TH3283 to TH4283, TH3284 to TH4284, TH3285 to TH4285, TH3286 to TH4286, TH3287 to TH4287, TH3288 to TH4288, TH3289 to TH4289, TH3290 to TH4290, TH3291 to TH4291, TH3292 to TH4292, TH3293 to TH4293, TH3294 to TH4294, TH3295 to TH4295, TH3296 to TH4296, TH3297 to TH4297, TH3298 to TH4298, TH3299 to TH4299, TH3300 to TH4300, TH3301 to TH4301, TH3302 to TH4302, TH3303 to TH4303, TH3304 to TH4304, TH3305 to TH4305, TH3306 to TH4306, TH3307 to TH4307, TH3308 to TH4308, TH3309 to TH4309, TH3310 to TH4310, TH3311 to TH4311, TH3312 to TH4312
