File: Prototype Schematics/inventeam_proto_schematics/inventeam_proto_schematics.kicad_sch (KiCad schematic)
At the start: 1 part, among them SW1 SW_Push_DPDT

Commit message: v16 minor 1
Parts:
- renumbered SW1 to SW1001
Other:
- sheet Thermistor Logic Schematic: file Matrix_Columns.kicad_sch -> Thermistor Logic Schematic.kicad_sch
- sheet Thermistor Matrix Schematic: file Thermistor_Matrix.kicad_sch -> Thermistor Matrix Schematic.kicad_sch
- title: Overview -> Root Schematic
Changed lines of the file:
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@@
 	(paper "User" 457.2 254)
 	(title_block
-		(title "Overview")
+		(title "Root Schematic")
 		(date "2025-10-26")
 		(rev "1/1/2026")
@@
 		(on_board yes)
 		(dnp no)
-		(property "Reference" "SW1"
+		(property "Reference" "SW1001"
 			(at 158.75 26.67 0)
 			(effects
@@
 			(project "Inventeam_Project_V3"
 				(path "/b2b47a1d-b0e5-4b64-b5c3-0417d2d1887a"
-					(reference "SW1")
+					(reference "SW1001")
 					(unit 1)
 				)
@@
 			)
 		)
-		(property "Sheetfile" "Matrix_Columns.kicad_sch"
+		(property "Sheetfile" "Thermistor Logic Schematic.kicad_sch"
 			(at 181.61 148.59 0)
 			(effects
@@
 			)
 		)
-		(property "Sheetfile" "Thermistor_Matrix.kicad_sch"
+		(property "Sheetfile" "Thermistor Matrix Schematic.kicad_sch"
 			(at 181.61 225.3746 0)
 			(effects

Commit message: V17
Connections:
- net FSR Logic Schematic/BAT+ renamed Logic Schematic (Pressure)/BAT+
- net FSR Logic Schematic/MCU_BAT+ renamed Logic Schematic (Pressure)/MCU_BAT+
Other:
- sheet Thermistor Logic Schematic renamed Logic Schematic (Temperature)
- removed sheet FSR Logic Schematic
- added sheet Logic Schematic (Pressure) (Logic Schematic.kicad_sch)
- sheet Logic Schematic (Temperature): file Thermistor Logic Schematic.kicad_sch -> Logic Schematic.kicad_sch
