File: PCB Final Schematic/inventeam_final_schematic/inventeam_final_schematic.kicad_sch (KiCad schematic)
At the start: 42 parts, among them J1 Conn_02x20_Top_Bottom, U1 OPA2333xxD, U11 MCP1525-TO, U2 MCP23S17_SP, U3 MCP23S17_SP, U4 TMUX1208PW, U7 TMUX1208PW

Commit message: Day 2 of PCB work
Parts:
- removed BT1: Battery, symbol Device:Battery
- removed JP1: SolderJumper_2_Open, symbol Jumper:SolderJumper_2_Open
- added F2: 2A, symbol Device:Polyfuse
- added H1, H2, H3, H4: Mounting Hole, symbol Mechanical:MountingHole_Pad
- added J2: Screw Terminal, symbol Connector:Screw_Terminal_01x02
- added J3: JST Male, symbol Connector_Generic:Conn_01x02
- added J4: JST Female, symbol Connector_Generic:Conn_01x02
- added J5: USB C, symbol Connector:USB_C_Receptacle_PowerOnly_6P
- added Q1, Q2: 2N3904, Package_TO_SOT_THT:TO-92_Inline, symbol Transistor_BJT:2N3904
- added Q3, Q4: SUP75P03-07-E3, symbol Transistor_FET:Q_PMOS_GDS
- added R19, R20: 5.1k, symbol Device:R_US
- added U5: LM393, symbol Comparator:LM393
- C12: value C_US -> 10uf
- C13: value C_US -> 0.1uf
- J1: value Conn_02x20_Top_Bottom -> Header
- R10, R11, R12, R13, R14, R15, R16, R17, R18, R7, R8, R9: value R_US -> 10k
Connections:
- net +3.3V: now also C13.1, U11.3 (Vin)
- net GND: now also C12.2, C13.2, R10.2, R11.2, R12.2, R13.2, R14.2, R15.2, R16.2, R17.2, R18.2, R7.2, R8.2, R9.2, U11.1 (Vss), H1.1, H2.1, H3.1, H4.1, J5.A12 (GND), J5.B12 (GND), J5.S1 (SHIELD), R19.2, R20.2
- net M1_ROW_10: now reaches R16.1
- net M1_ROW_10: now also J1.35 (Pin_35), U4.5 (S2)
- net M1_ROW_1: now reaches R7.1
- net M1_ROW_1: now also J1.17 (Pin_17), U7.4 (S1)
- net M1_ROW_2: now reaches J1.18 (Pin_18)
- net M1_ROW_2: now also R8.1, U7.5 (S2)
- net M1_ROW_3: now reaches J1.19 (Pin_19)
- net M1_ROW_3: now also R9.1, U7.6 (S3)
- net M1_ROW_4: now reaches J1.20 (Pin_20)
- net M1_ROW_4: now also R10.1, U7.7 (S4)
- net M1_ROW_12: now reaches J1.33 (Pin_33)
- net M1_ROW_12: now also R18.1, U4.7 (S4)
- net M1_ROW_11: now reaches J1.34 (Pin_34)
- net M1_ROW_11: now also R17.1, U4.6 (S3)
- net M1_ROW_9: now reaches J1.36 (Pin_36)
- net M1_ROW_9: now also R15.1, U4.4 (S1)
- net M1_ROW_8: now reaches J1.37 (Pin_37)
- net M1_ROW_8: now also R14.1, U7.9 (S8)
- net M1_ROW_7: now reaches J1.38 (Pin_38)
- net M1_ROW_7: now also R13.1, U7.10 (S7)
- net M1_ROW_6: now reaches J1.39 (Pin_39)
- net M1_ROW_5: now reaches J1.40 (Pin_40)
- net M1_ROW_5: now also R11.1, R12.1, U7.11 (S6), U7.12 (S5)
- net M1_GPIO_14: now reaches U7.1 (A0)
- net M1_GPIO_14: now also A1.19 (A6/IO14), U4.1 (A0)
- net M1_GPIO_15: now reaches U7.15 (A2)
- net M1_GPIO_15: now also A1.21 (A8/IO15), U4.15 (A2)
- net M1_GPIO_32: now reaches U7.16 (A1)
- net M1_GPIO_32: now also A1.20 (A7/IO32), U4.16 (A1)
- net M1_GPIO_33: now reaches U7.2 (EN)
- net M1_GPIO_33: now also A1.22 (A9/IO33)
- net at U11.2 (Vout): now also C12.1, U4.9 (S8)
- net M1_GPIO_27: now reaches U4.2 (EN)
- net M1_GPIO_27: now also A1.23 (A10/IO27)
- net M2_TX: now reaches A1.14 (RX/IO16)
- net M1_TX: now reaches A1.15 (TX/IO17)
- new net: J2.1 (Pin_1), J3.2 (Pin_2)
- new net: J2.2 (Pin_2), J4.1 (Pin_1)
- new net: J3.1 (Pin_1), J4.2 (Pin_2)
- new net: F2.2, J5.A9 (VBUS), J5.B9 (VBUS)
- new net +5V: F2.1
- new net CC1: J5.A5 (CC1), R19.1
- new net CC2: J5.B5 (CC2), R20.1
- no-connect marks 12 -> 25
Other:
- note added: "Battery"
- note added: "Circuit Universal Power Input"
- note added: "Column & Row External connector"
- note added: "Column Output"
- note added: "Microcontroller"
- note added: "Row Input"
- note added: "Row input buffers"
- note removed: "Matrix Logic 2"
- moved on the sheet: A1, C1, C10, C11, C12, C13, C2, C3, C4, C5, C6, C7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

Commit message: Finished USB C input
Parts:
- removed Q1, Q2: 2N3904, Package_TO_SOT_THT:TO-92_Inline, symbol Transistor_BJT:2N3904
- removed Q3, Q4: SUP75P03-07-E3, symbol Transistor_FET:Q_PMOS_GDS
- removed U5: LM393, symbol Comparator:LM393
- added C15: 47uf, symbol Device:C_US
- added D1: 1.5KE6.8A, symbol Device:D_TVS
- added D2: SMF3.3A, symbol Device:D_TVS
- added U6, U8: LM66100DCK, Package_TO_SOT_SMD:SOT-363_SC-70-6, symbol Power_Management:LM66100DCK
- J5: value USB C -> USB_C_Receptacle_PowerOnly_6P
Connections:
- net +3.3V: now also D2.2 (A2)
- net +5V: now also D1.1 (A1), U6.1 (VIN), U8.1 (VIN)
- net GND: now also C15.2, D1.2 (A2), D2.1 (A1), U6.2 (GND), U6.3 (~{CE}), U8.2 (GND), U8.3 (~{CE})
- net M1_VBUS: now also A1.26 (USB), U6.6 (VOUT)
- net M2_VBUS: now also U8.6 (VOUT)
- net at F2.2, J5.A9 (VBUS), J5.B9 (VBUS): now also C15.1
- net CC1: no longer names the net of J5.A5 (CC1), R19.1
- net CC2: no longer names the net of J5.B5 (CC2), R20.1
- no-connect marks 25 -> 26
Other:
- note added: "More than one USB must never be used on the board at once."
- moved on the sheet: A1, C1, C2, C3, C4, C5, F1, F2, H1, H2, H3, H4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

Commit message: Logic PCB V1
Parts:
- added A2: Adafruit_Feather_HUZZAH32_ESP32, Module:Adafruit_Feather, symbol MCU_Module:Adafruit_Feather_HUZZAH32_ESP32
- added C15, C17, C18, C21, C22, C23, C25, C26, C27: 0.1uf, symbol Device:C_US
- added C16, C19: 1nf, symbol Device:C_US
- added C20, C24: 10uf, symbol Device:C_US
- added D3: SMF3.3A, symbol Device:D_TVS
- added F3: 1A, symbol Device:Polyfuse
- added J6: Header, symbol Connector_Generic:Conn_02x20_Top_Bottom
- added J7: Screw Terminal, symbol Connector:Screw_Terminal_01x02
- added J8: JST Female, symbol Connector_Generic:Conn_01x02
- added J9: JST Male, symbol Connector_Generic:Conn_01x02
- added R21, R22, R23, R25, R26, R28, R29, R30, R31, R32, R34, R36: 10k, symbol Device:R_US
- added R24, R33: 220, symbol Device:R_US
- added R27, R35: 1M, symbol Device:R_US
- added R37, R38: 1k, symbol Device:R_US
- added TP1, TP10, TP11, TP12, TP13, TP14, TP15, TP16, TP17, TP18, TP19, TP2, TP20, TP21, TP22, TP23, TP24, TP25, TP26, TP27, TP28, TP29, TP3, TP30, TP31, TP32, TP33, TP34, TP4, TP5, TP6, TP7, TP8, TP9: TestPoint_Probe, symbol Connector:TestPoint_Probe
- added U10, U11: TMUX1208PW, Package_SO:TSSOP-16_4.4x5mm_P0.65mm, symbol Analog_Switch:TMUX1208PW
- added U12, U9: MCP23S17_SP, Package_DIP:DIP-28_W7.62mm, symbol Interface_Expansion:MCP23S17_SP
- added U13: MCP1525-TO, Package_TO_SOT_THT:TO-92_Inline, symbol Reference_Voltage:MCP1525-TO
- added U14: OPA2333xxD, symbol Amplifier_Operational:OPA2333xxD
- renumbered C8 to C1, C3 to C10, C1 to C11, C4 to C12, C5 to C13, C2 to C14, C9 to C2, C6 to C3, C10 to C4, C11 to C5, C15 to C6, C12 to C7, C7 to C8, C13 to C9, F2 to F1, F1 to F2, H3 to H2, H2 to H3, J5 to J2, J2 to J3, J3 to J5, R7 to R1, R14 to R10, R15 to R11, R16 to R12, R5 to R13, R19 to R14, R20 to R15, R17 to R16, R6 to R17, R1 to R19, R8 to R2, R2 to R20, R9 to R3, R3 to R4, R10 to R5, R11 to R6, R4 to R7, R12 to R8, R13 to R9, U3 to U1, U7 to U2, U4 to U3, U2 to U4, U6 to U5, U8 to U6, U11 to U7, U1 to U8
Connections:
- net +5V: now also TP6.1
- net GND: now also U5.5 (ST), U6.5 (ST), A2.16 (IO21), A2.4 (GND), A2.6 (DAC1/A1), C15.2, C16.2, C17.2, C18.2, C19.2, C20.2, C21.2, C22.2, C23.2, C24.2, C25.2, C26.2, C27.2, D3.1 (A1), R21.2, R22.2, R23.2, R25.2, R26.2, R27.2, R28.2, R29.2, R30.2, R31.2, R32.2, R34.2, R35.2, R36.2, TP13.1, TP29.1, TP4.1, U10.14 (GND), U10.3 (VSS), U11.14 (GND), U11.3 (VSS), U12.10 (VSS), U12.15 (A0), U12.16 (A1), U12.17 (A2), U13.1 (Vss), U14.4 (V-), U9.10 (VSS), U9.15 (A0), U9.16 (A1), U9.17 (A2)
- net M1_A2: now also TP14.1, TP17.1
- net M1_A3: now also TP15.1, TP18.1
- net M1_GPIO_12: now also TP3.1
- net M1_GPIO_13: now also TP10.1
- net M1_GPIO_18: now also TP12.1
- net M1_GPIO_19: now also TP2.1, TP8.1
- net M1_GPIO_5: now also TP11.1
- net M1_NON_IN_1: now also TP1.1
- net M1_NON_IN_2: now also TP5.1
- net M1_ROW_5: no longer R8.1, U2.11 (S6)
- net M1_ROW_6: now also R8.1, U2.11 (S6)
- net M1_TX: now also A2.14 (RX/IO16)
- net M2_TX: now also A2.15 (TX/IO17)
- net M2_VBUS: now also A2.26 (USB)
- net at J3.2 (Pin_2), J4.1 (Pin_1): now also TP7.1
- net at C7.1, U3.9 (S8), U7.2 (Vout): now also TP9.1
- net +3.3V renamed M1_3.3V
- net M1_3.3V: now also TP16.1
- new net: R38.1, U14.6 (-), U14.7
- new net: R33.2, R35.1, U11.8 (D)
- new net: A2.2 (3V3), C24.1, F3.1
- new net: R24.2, R27.1, U10.8 (D)
- new net: C20.1, TP25.1, U11.9 (S8), U13.2 (Vout)
- new net: R37.1, U14.1, U14.2 (-)
- new net: J7.2 (Pin_2), J8.1 (Pin_1), TP23.1
- new net: J8.2 (Pin_2), J9.1 (Pin_1)
- new net: J7.1 (Pin_1), J9.2 (Pin_2)
- new net M2_3.3V: C15.1, C17.1, C18.1, C21.1, C22.1, C23.1, C27.1, D3.2 (A2), F3.2, TP32.1, U10.13 (VDD), U11.13 (VDD), U12.18 (~{RESET}), U12.9 (VDD), U13.3 (Vin), U14.8 (V+), U9.18 (~{RESET}), U9.9 (VDD)
- new net M2_A2: A2.7 (I34/A2), C25.1, R37.2, TP30.1, TP33.1
- new net M2_A3: A2.8 (I39/A3), C26.1, R38.2, TP31.1, TP34.1
- new net M2_COL_1: J6.5 (Pin_5), U9.28 (GPA7)
- new net M2_COL_10: J6.23 (Pin_23), U9.7 (GPB6)
- new net M2_COL_11: J6.22 (Pin_22), U9.6 (GPB5)
- new net M2_COL_12: J6.21 (Pin_21), U9.5 (GPB4)
- new net M2_COL_13: J6.4 (Pin_4), U9.4 (GPB3)
- new net M2_COL_14: J6.3 (Pin_3), U9.3 (GPB2)
- new net M2_COL_15: J6.2 (Pin_2), U9.2 (GPB1)
- new net M2_COL_16: J6.1 (Pin_1), U9.1 (GPB0)
- new net M2_COL_17: J6.16 (Pin_16), U12.28 (GPA7)
- new net M2_COL_18: J6.15 (Pin_15), U12.27 (GPA6)
- new net M2_COL_19: J6.14 (Pin_14), U12.26 (GPA5)
- new net M2_COL_2: J6.6 (Pin_6), U9.27 (GPA6)
- new net M2_COL_20: J6.13 (Pin_13), U12.25 (GPA4)
- new net M2_COL_21: J6.30 (Pin_30), U12.6 (GPB5)
- new net M2_COL_22: J6.29 (Pin_29), U12.5 (GPB4)
- new net M2_COL_23: J6.9 (Pin_9), U12.4 (GPB3)
- new net M2_COL_24: J6.10 (Pin_10), U12.3 (GPB2)
- new net M2_COL_25: J6.11 (Pin_11), U12.2 (GPB1)
- new net M2_COL_26: J6.12 (Pin_12), U12.1 (GPB0)
- new net M2_COL_3: J6.7 (Pin_7), U9.26 (GPA5)
- new net M2_COL_4: J6.8 (Pin_8), U9.25 (GPA4)
- new net M2_COL_5: J6.25 (Pin_25), U9.24 (GPA3)
- new net M2_COL_6: J6.26 (Pin_26), U9.23 (GPA2)
- new net M2_COL_7: J6.27 (Pin_27), U9.22 (GPA1)
- new net M2_COL_8: J6.28 (Pin_28), U9.21 (GPA0)
- new net M2_COL_9: J6.24 (Pin_24), U9.8 (GPB7)
- new net M2_GPIO_12: A2.24 (A11/IO12), TP21.1, U9.11 (~{CS})
- new net M2_GPIO_13: A2.25 (A12/IO13), TP26.1, U12.11 (~{CS})
- new net M2_GPIO_14: A2.19 (A6/IO14), U10.1 (A0), U11.1 (A0)
- new net M2_GPIO_15: A2.21 (A8/IO15), U10.15 (A2), U11.15 (A2)
- new net M2_GPIO_18: A2.12 (MOSI/IO18), TP28.1, U12.13 (SI), U9.13 (SI)
- new net M2_GPIO_19: A2.13 (MISO/IO19), TP20.1, TP24.1, U12.14 (SO), U9.14 (SO)
- new net M2_GPIO_27: A2.23 (A10/IO27), U11.2 (EN)
- new net M2_GPIO_32: A2.20 (A7/IO32), U10.16 (A1), U11.16 (A1)
- new net M2_GPIO_33: A2.22 (A9/IO33), U10.2 (EN)
- new net M2_GPIO_5: A2.11 (SCK/IO5), TP27.1, U12.12 (SCK), U9.12 (SCK)
- new net M2_NON_IN_1: C16.1, R24.1, TP19.1, U14.3 (+)
- new net M2_NON_IN_2: C19.1, R33.1, TP22.1, U14.5 (+)
- new net M2_ROW_1: J6.17 (Pin_17), R21.1, U10.4 (S1)
- new net M2_ROW_10: J6.35 (Pin_35), R32.1, U11.5 (S2)
- new net M2_ROW_11: J6.34 (Pin_34), R34.1, U11.6 (S3)
- new net M2_ROW_12: J6.33 (Pin_33), R36.1, U11.7 (S4)
- new net M2_ROW_2: J6.18 (Pin_18), R22.1, U10.5 (S2)
- new net M2_ROW_3: J6.19 (Pin_19), R23.1, U10.6 (S3)
- new net M2_ROW_4: J6.20 (Pin_20), R25.1, U10.7 (S4)
- new net M2_ROW_5: J6.40 (Pin_40), R26.1, U10.12 (S5)
- new net M2_ROW_6: J6.39 (Pin_39), R28.1, U10.11 (S6)
- new net M2_ROW_7: J6.38 (Pin_38), R29.1, U10.10 (S7)
- new net M2_ROW_8: J6.37 (Pin_37), R30.1, U10.9 (S8)
- new net M2_ROW_9: J6.36 (Pin_36), R31.1, U11.4 (S1)
- no-connect marks 26 -> 47
Other:
- note added: "Matrix Logic 2"
- moved on the sheet: C6, D1, F1, H1, H2, H3, H4, J2, J4, J5, R14, R15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

Commit message: V1 minor 1
Parts:
- removed J3, J7: Screw Terminal, symbol Connector:Screw_Terminal_01x02
- added J3: Screw_Terminal_01x04, symbol Connector:Screw_Terminal_01x04
- C1, C10, C11, C12, C13, C14, C15, C17, C18, C20, C21, C22, C23, C24, C25, C26, C27, C3, C4, C7, C8, C9: footprint (none) -> Capacitor_THT:CP_Radial_D5.0mm_P2.50mm
- C16, C19, C2, C5: footprint (none) -> Capacitor_THT:CP_Axial_L10.0mm_D4.5mm_P15.00mm_Horizontal
- H1, H2, H3, H4: footprint (none) -> MountingHole:MountingHole_2.5mm_Pad
- R1, R10, R11, R12, R16, R17, R18, R19, R2, R20, R21, R22, R23, R25, R26, R27, R28, R29, R3, R30, R31, R32, R34, R35, R36, R37, R38, R5, R6, R7, R8, R9: footprint (none) -> Resistor_THT:R_Axial_DIN0207_L6.3mm_D2.5mm_P7.62mm_Horizontal
- TP1, TP10, TP11, TP12, TP13, TP14, TP15, TP16, TP17, TP18, TP19, TP2, TP20, TP21, TP22, TP23, TP24, TP25, TP26, TP27, TP28, TP29, TP3, TP30, TP31, TP32, TP33, TP34, TP4, TP5, TP6, TP7, TP8, TP9: footprint (none) -> TestPoint:TestPoint_Pad_D1.0mm
- U14, U8: footprint (none) -> Package_SO:SOIC-8_3.9x4.9mm_P1.27mm
Connections:
- net at J4.1 (Pin_1), TP7.1: now also J3.4 (Pin_4)
- net at J5.2 (Pin_2): now also J3.3 (Pin_3)
- net at J8.1 (Pin_1), TP23.1: now also J3.2 (Pin_2)
- net at J9.2 (Pin_2): now also J3.1 (Pin_1)
Other:
- note added: "Battery connections"
- note removed: "Battery"
- moved on the sheet: C6, D1, F1, H1, H2, H3, H4, J1, J2, J4, J5, J6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
