File: Finalized Logic Schematic/inventeam_final_schematic/inventeam_final_schematic.kicad_sch (KiCad schematic)
At the start: 133 parts, among them J1 Header, J2 USB_C_Receptacle_PowerOnly_6P, J3 Screw_Terminal_01x04, J4 JST Female, J5 JST Male, J6 Header, J8 JST Female, J9 JST Male, U1 MCP23S17_SP, U10 TMUX1208PW, U11 TMUX1208PW, U12 MCP23S17_SP, U13 MCP1525-TO, U14 OPA2333xxD, U2 TMUX1208PW, U3 TMUX1208PW, U4 MCP23S17_SP, U5 LM66100DCK, U6 LM66100DCK, U7 MCP1525-TO, U8 OPA2333xxD, U9 MCP23S17_SP

Commit message: Prepare for finalized matrix
Parts:
- D1: footprint (none) -> Diode_THT:D_DO-201_P15.24mm_Horizontal
- D2, D3: footprint (none) -> Diode_SMD:D_SOD-123F
- J3: footprint (none) -> TerminalBlock:TerminalBlock_Xinya_XY308-2.54-4P_1x04_P2.54mm_Horizontal
- R13, R24, R33, R4: footprint (none) -> Resistor_THT:R_Axial_DIN0207_L6.3mm_D2.5mm_P10.16mm_Horizontal
Changed lines of the file:
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@@
 			)
 		)
-		(property "Footprint" ""
+		(property "Footprint" "Resistor_THT:R_Axial_DIN0207_L6.3mm_D2.5mm_P10.16mm_Horizontal"
 			(at 432.054 183.134 90)
 			(effects
@@
 			)
 		)
-		(property "Footprint" ""
+		(property "Footprint" "Resistor_THT:R_Axial_DIN0207_L6.3mm_D2.5mm_P10.16mm_Horizontal"
 			(at 142.494 183.134 90)
 			(effects
@@
 			)
 		)
-		(property "Footprint" ""
+		(property "Footprint" "Diode_SMD:D_SOD-123F"
 			(at 287.02 255.27 0)
 			(effects
@@
 			)
 		)
-		(property "Footprint" ""
+		(property "Footprint" "Diode_THT:D_DO-201_P15.24mm_Horizontal"
 			(at 76.2 412.75 0)
 			(effects
@@
 			)
 		)
-		(property "Footprint" ""
+		(property "Footprint" "TerminalBlock:TerminalBlock_Xinya_XY308-2.54-4P_1x04_P2.54mm_Horizontal"
 			(at 229.87 426.72 0)
 			(effects
@@
 			)
 		)
-		(property "Footprint" ""
+		(property "Footprint" "Resistor_THT:R_Axial_DIN0207_L6.3mm_D2.5mm_P10.16mm_Horizontal"
 			(at 358.394 183.134 90)
 			(effects
@@
 			)
 		)
-		(property "Footprint" ""
+		(property "Footprint" "Resistor_THT:R_Axial_DIN0207_L6.3mm_D2.5mm_P10.16mm_Horizontal"
 			(at 68.834 183.134 90)
 			(effects
@@
 			)
 		)
-		(property "Footprint" ""
+		(property "Footprint" "Diode_SMD:D_SOD-123F"
 			(at 576.58 255.27 0)
 			(effects
