File: Finalized Logic Schematic/inventeam_final_schematic/inventeam_final_schematic.kicad_sch (KiCad schematic)
At the start: 133 parts, among them J1 Header, J2 USB_C_Receptacle_PowerOnly_6P, J3 Screw_Terminal_01x04, J4 JST Female, J5 JST Male, J6 Header, J8 JST Female, J9 JST Male, U1 MCP23S17_SP, U10 TMUX1208PW, U11 TMUX1208PW, U12 MCP23S17_SP, U13 MCP1525-TO, U14 OPA2333xxD, U2 TMUX1208PW, U3 TMUX1208PW, U4 MCP23S17_SP, U5 LM66100DCK, U6 LM66100DCK, U7 MCP1525-TO, U8 OPA2333xxD, U9 MCP23S17_SP

Commit message: Logic schematic v1.3
Parts:
- removed J1, J6: Header, symbol Connector_Generic:Conn_02x20_Top_Bottom
- added C3: 0.1uf, Capacitor_THT:CP_Radial_D5.0mm_P2.50mm, symbol Device:C_US
- added J2, J8: Conn_02x20_Odd_Even, Connector_PinHeader_2.54mm:PinHeader_2x20_P2.54mm_Vertical, symbol Connector_Generic:Conn_02x20_Odd_Even
- C4: renamed from C6; footprint (none) -> Capacitor_THT:CP_Radial_D5.0mm_P2.50mm
- F1: value 2A -> 1A; footprint (none) -> Fuse:Fuse_BelFuse_0ZRE0100FF_L18.7mm_W5.1mm
- F2, F3: footprint (none) -> Fuse:Fuse_BelFuse_0ZRE0100FF_L18.7mm_W5.1mm
- J1: renamed from J2; footprint (none) -> Connector_USB:USB_C_Receptacle_GCT_USB4125-xx-x_6P_TopMnt_Horizontal
- J4, J5: footprint (none) -> Connector_PinHeader_2.54mm:PinHeader_1x02_P2.54mm_Vertical
- J6: renamed from J8; footprint (none) -> Connector_PinHeader_2.54mm:PinHeader_1x02_P2.54mm_Vertical
- J7: renamed from J9; footprint (none) -> Connector_PinHeader_2.54mm:PinHeader_1x02_P2.54mm_Vertical
- R6: renamed from R14; footprint (none) -> Resistor_THT:R_Axial_DIN0207_L6.3mm_D2.5mm_P7.62mm_Horizontal
- R7: renamed from R15; footprint (none) -> Resistor_THT:R_Axial_DIN0207_L6.3mm_D2.5mm_P7.62mm_Horizontal
- renumbered C9 to C10, C10 to C11, C11 to C12, C12 to C13, C13 to C14, C14 to C15, C15 to C16, C16 to C17, C17 to C18, C18 to C19, C19 to C20, C20 to C21, C21 to C22, C22 to C23, C23 to C24, C24 to C25, C25 to C26, C26 to C27, C27 to C28, C3 to C5, C4 to C6, C5 to C7, C7 to C8, C8 to C9, R8 to R10, R9 to R11, R10 to R12, R11 to R13, R12 to R14, R13 to R15, R6 to R8, R7 to R9, TP4 to TP1, TP11 to TP10, TP12 to TP11, TP7 to TP12, TP23 to TP13, TP13 to TP14, TP14 to TP15, TP15 to TP16, TP16 to TP17, TP17 to TP18, TP18 to TP19, TP1 to TP2, TP19 to TP20, TP20 to TP21, TP21 to TP22, TP22 to TP23, TP6 to TP3, TP2 to TP4, TP3 to TP5, TP5 to TP6, TP8 to TP7, TP9 to TP8, TP10 to TP9, U5 to U3, U6 to U4, U3 to U5, U4 to U6
Connections:
- net +5V: now also C3.1
- net GND: now also C3.2, J2.24 (Pin_24), J8.24 (Pin_24)
- net M1_COL_1: now also J2.9 (Pin_9)
- net M1_COL_10: now also J2.6 (Pin_6)
- net M1_COL_11: now also J2.4 (Pin_4)
- net M1_COL_12: now also J2.2 (Pin_2)
- net M1_COL_13: now also J2.7 (Pin_7)
- net M1_COL_14: now also J2.5 (Pin_5)
- net M1_COL_15: now also J2.3 (Pin_3)
- net M1_COL_16: now also J2.1 (Pin_1)
- net M1_COL_17: now also J2.31 (Pin_31)
- net M1_COL_18: now also J2.29 (Pin_29)
- net M1_COL_19: now also J2.27 (Pin_27)
- net M1_COL_2: now also J2.11 (Pin_11)
- net M1_COL_20: now also J2.25 (Pin_25)
- net M1_COL_21: now also J2.20 (Pin_20)
- net M1_COL_22: now also J2.18 (Pin_18)
- net M1_COL_23: now also J2.17 (Pin_17)
- net M1_COL_24: now also J2.19 (Pin_19)
- net M1_COL_25: now also J2.21 (Pin_21)
- net M1_COL_26: now also J2.23 (Pin_23)
- net M1_COL_3: now also J2.13 (Pin_13)
- net M1_COL_4: now also J2.15 (Pin_15)
- net M1_COL_5: now also J2.10 (Pin_10)
- net M1_COL_6: now also J2.12 (Pin_12)
- net M1_COL_7: now also J2.14 (Pin_14)
- net M1_COL_8: now also J2.16 (Pin_16)
- net M1_COL_9: now also J2.8 (Pin_8)
- net M1_ROW_1: now also J2.33 (Pin_33)
- net M1_ROW_10: now also J2.30 (Pin_30)
- net M1_ROW_11: now also J2.28 (Pin_28)
- net M1_ROW_12: now also J2.26 (Pin_26)
- net M1_ROW_2: now also J2.35 (Pin_35)
- net M1_ROW_3: now also J2.37 (Pin_37)
- net M1_ROW_4: now also J2.39 (Pin_39)
- net M1_ROW_5: now also J2.40 (Pin_40)
- net M1_ROW_6: now also J2.38 (Pin_38)
- net M1_ROW_7: now also J2.36 (Pin_36)
- net M1_ROW_8: now also J2.34 (Pin_34)
- net M1_ROW_9: now also J2.32 (Pin_32)
- net M2_COL_1: now also J8.9 (Pin_9)
- net M2_COL_10: now also J8.6 (Pin_6)
- net M2_COL_11: now also J8.4 (Pin_4)
- net M2_COL_12: now also J8.2 (Pin_2)
- net M2_COL_13: now also J8.7 (Pin_7)
- net M2_COL_14: now also J8.5 (Pin_5)
- net M2_COL_15: now also J8.3 (Pin_3)
- net M2_COL_16: now also J8.1 (Pin_1)
- net M2_COL_17: now also J8.31 (Pin_31)
- net M2_COL_18: now also J8.29 (Pin_29)
- net M2_COL_19: now also J8.27 (Pin_27)
- net M2_COL_2: now also J8.11 (Pin_11)
- net M2_COL_20: now also J8.25 (Pin_25)
- net M2_COL_21: now also J8.20 (Pin_20)
- net M2_COL_22: now also J8.18 (Pin_18)
- net M2_COL_23: now also J8.17 (Pin_17)
- net M2_COL_24: now also J8.19 (Pin_19)
- net M2_COL_25: now also J8.21 (Pin_21)
- net M2_COL_26: now also J8.23 (Pin_23)
- net M2_COL_3: now also J8.13 (Pin_13)
- net M2_COL_4: now also J8.15 (Pin_15)
- net M2_COL_5: now also J8.10 (Pin_10)
- net M2_COL_6: now also J8.12 (Pin_12)
- net M2_COL_7: now also J8.14 (Pin_14)
- net M2_COL_8: now also J8.16 (Pin_16)
- net M2_COL_9: now also J8.8 (Pin_8)
- net M2_ROW_1: now also J8.33 (Pin_33)
- net M2_ROW_10: now also J8.30 (Pin_30)
- net M2_ROW_11: now also J8.28 (Pin_28)
- net M2_ROW_12: now also J8.26 (Pin_26)
- net M2_ROW_2: now also J8.35 (Pin_35)
- net M2_ROW_3: now also J8.37 (Pin_37)
- net M2_ROW_4: now also J8.39 (Pin_39)
- net M2_ROW_5: now also J8.40 (Pin_40)
- net M2_ROW_6: now also J8.38 (Pin_38)
- net M2_ROW_7: now also J8.36 (Pin_36)
- net M2_ROW_8: now also J8.34 (Pin_34)
- net M2_ROW_9: now also J8.32 (Pin_32)
Other:
- note added: "Matrix Logic 1 (Temperature)"
- note added: "Matrix Logic 2 (Pressure)"
- note removed: "Matrix Logic 1"
- note removed: "Matrix Logic 2"
- moved on the sheet: D1

Commit message: Logic schematic v1.4
Parts:
- added J2: Conn_01x02, Connector_PinHeader_2.54mm:PinHeader_1x02_P2.54mm_Vertical, symbol Connector_Generic:Conn_01x02
- C1, C10, C11, C13, C14, C15, C16, C18, C19, C22, C23, C24, C26, C27, C28, C3, C5, C6, C9: footprint Capacitor_THT:CP_Radial_D5.0mm_P2.50mm -> Capacitor_THT:C_Disc_D5.0mm_W2.5mm_P5.00mm
- C12, C21, C25, C8: footprint Capacitor_THT:CP_Radial_D5.0mm_P2.50mm -> Capacitor_THT:C_Disc_D5.0mm_W2.5mm_P2.50mm
- F1, F2, F3: footprint Fuse:Fuse_BelFuse_0ZRE0100FF_L18.7mm_W5.1mm -> X16_GF100_PPTC:X16 GF100
- renumbered J2 to J3, J3 to J4, J4 to J5, J5 to J6, J6 to J7, J7 to J8, J8 to J9, R7 to R4, R6 to R5, R4 to R6, R5 to R7
Connections:
- net GND: now also J2.2 (Pin_2)
- net at C4.1, F1.2, J1.A9 (VBUS)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: now also J2.1 (Pin_1)
Other:
- moved on the sheet: C3, C4, D1, F1, H1, H2, H3, H4, J1, J4, J5, J6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

Commit message: Logic schematic V1.4+
Parts:
- added C10, C11: 1uf, symbol Device:C_Polarized_US
- added C7, C8: 0.1uf, symbol Device:C_US
- renumbered C8 to C12, C9 to C13, C10 to C14, C11 to C15, C12 to C16, C13 to C17, C14 to C18, C15 to C19, C16 to C20, C17 to C21, C18 to C22, C19 to C23, C20 to C24, C21 to C25, C22 to C26, C23 to C27, C24 to C28, C25 to C29, C26 to C30, C27 to C31, C28 to C32, C7 to C9, R6 to R5, R5 to R6, TP14 to TP12, TP15 to TP13, TP16 to TP14, TP17 to TP15, TP18 to TP16, TP19 to TP17, TP12 to TP18, TP13 to TP19, TP4 to TP3, TP3 to TP4, U5 to U3, U6 to U4, U3 to U5, U4 to U6
Connections:
- net +5V: now also C10.1, C11.1, C7.1, C8.1
- net GND: now also C10.2, C11.2, C7.2, C8.2
Other:
- moved on the sheet: C3, C4, D1, F1, H1, H2, H3, H4, J1, J2, J4, J5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

Commit message: Removed extra 0.1uf capacitor
Parts:
- removed C3: 0.1uf, Capacitor_THT:C_Disc_D5.0mm_W2.5mm_P5.00mm, symbol Device:C_US
- C10: renamed from C11; footprint (none) -> Capacitor_THT:CP_Axial_L10.0mm_D4.5mm_P15.00mm_Horizontal
- C6: renamed from C7; footprint (none) -> Capacitor_THT:C_Disc_D5.0mm_W2.5mm_P5.00mm
- C7: renamed from C8; footprint (none) -> Capacitor_THT:C_Disc_D5.0mm_W2.5mm_P5.00mm
- C9: renamed from C10; footprint (none) -> Capacitor_THT:CP_Axial_L10.0mm_D4.5mm_P15.00mm_Horizontal
- renumbered C12 to C11, C13 to C12, C14 to C13, C15 to C14, C16 to C15, C17 to C16, C18 to C17, C19 to C18, C20 to C19, C21 to C20, C22 to C21, C23 to C22, C24 to C23, C25 to C24, C26 to C25, C27 to C26, C28 to C27, C29 to C28, C30 to C29, C4 to C3, C31 to C30, C32 to C31, C5 to C4, C6 to C5, C9 to C8
Other:
- moved on the sheet: D1, F1
