File: Finalized Logic Schematic/inventeam_final_schematic/inventeam_final_schematic.kicad_pcb (KiCad board)
At the start: 2 copper layers, 135 parts, among them J1 USB_C_Receptacle_PowerOnly_6P, J2 Conn_01x02, J3 Conn_02x20_Odd_Even, J4 Screw_Terminal_01x04, J5 JST Female, J6 JST Male, J7 JST Female, J8 JST Male, J9 Conn_02x20_Odd_Even, U1 MCP23S17_SP, U10 TMUX1208PW, U11 TMUX1208PW, U12 MCP23S17_SP, U13 MCP1525-TO, U14 OPA2333xxD, U2 TMUX1208PW, U3 LM66100DCK, U4 LM66100DCK, U5 TMUX1208PW, U6 MCP23S17_SP, U7 MCP1525-TO, U8 OPA2333xxD, U9 MCP23S17_SP

Commit message: Logic schematic V1.4+
Parts:
- removed C10, C11: 0.1uf, Capacitor_THT:C_Disc_D5.0mm_W2.5mm_P5.00mm
- removed C7: 1nf, Capacitor_THT:CP_Axial_L10.0mm_D4.5mm_P15.00mm_Horizontal
- removed C8: 10uf, Capacitor_THT:C_Disc_D5.0mm_W2.5mm_P2.50mm
- added C29: 10uf, Capacitor_THT:C_Disc_D5.0mm_W2.5mm_P2.50mm, F.Cu at (446.3, 162.0)
- added C30: 0.1uf, Capacitor_THT:C_Disc_D5.0mm_W2.5mm_P5.00mm, F.Cu at (430.3, 108.2)
- added C31: 0.1uf, Capacitor_THT:C_Disc_D5.0mm_W2.5mm_P5.00mm, F.Cu at (430.3, 112.3)
- added C32: 0.1uf, Capacitor_THT:C_Disc_D5.0mm_W2.5mm_P5.00mm, F.Cu at (430.3, 116.3)
- C16: value 0.1uf -> 10uf; footprint Capacitor_THT:C_Disc_D5.0mm_W2.5mm_P5.00mm -> Capacitor_THT:C_Disc_D5.0mm_W2.5mm_P2.50mm
- C17, C20: value 1nf -> 0.1uf; footprint Capacitor_THT:CP_Axial_L10.0mm_D4.5mm_P15.00mm_Horizontal -> Capacitor_THT:C_Disc_D5.0mm_W2.5mm_P5.00mm
- C21: value 10uf -> 1nf; footprint Capacitor_THT:C_Disc_D5.0mm_W2.5mm_P2.50mm -> Capacitor_THT:CP_Axial_L10.0mm_D4.5mm_P15.00mm_Horizontal
- C24, C9: value 0.1uf -> 1nf; footprint Capacitor_THT:C_Disc_D5.0mm_W2.5mm_P5.00mm -> Capacitor_THT:CP_Axial_L10.0mm_D4.5mm_P15.00mm_Horizontal
- R5: value 5.1k -> 220; footprint Resistor_THT:R_Axial_DIN0207_L6.3mm_D2.5mm_P7.62mm_Horizontal -> Resistor_THT:R_Axial_DIN0207_L6.3mm_D2.5mm_P10.16mm_Horizontal
- R6: value 220 -> 5.1k; footprint Resistor_THT:R_Axial_DIN0207_L6.3mm_D2.5mm_P10.16mm_Horizontal -> Resistor_THT:R_Axial_DIN0207_L6.3mm_D2.5mm_P7.62mm_Horizontal
- U3: value LM66100DCK -> TMUX1208PW; footprint Package_TO_SOT_SMD:SOT-363_SC-70-6 -> Package_SO:TSSOP-16_4.4x5mm_P0.65mm
- U4: value LM66100DCK -> MCP23S17_SP; footprint Package_TO_SOT_SMD:SOT-363_SC-70-6 -> Package_DIP:DIP-28_W7.62mm
- U5: value TMUX1208PW -> LM66100DCK; footprint Package_SO:TSSOP-16_4.4x5mm_P0.65mm -> Package_TO_SOT_SMD:SOT-363_SC-70-6
- U6: value MCP23S17_SP -> LM66100DCK; footprint Package_DIP:DIP-28_W7.62mm -> Package_TO_SOT_SMD:SOT-363_SC-70-6
- moved R5 115.1 mm to (432.6, 149.8)
- moved U6 94.2 mm to (395.1, 157.0)
- moved C16 87.7 mm to (446.3, 153.9)
- moved U3 85.3 mm to (441.6, 108.0)
- moved C24 70.6 mm to (414.2, 149.5)
- moved U5 68.4 mm to (395.1, 153.1)
- moved C9 55.8 mm to (414.2, 136.5)
- moved C23 50.9 mm to (422.2, 120.4)
- moved C17 48.3 mm to (422.2, 100.1)
- moved R6 47.6 mm to (399.7, 79.9)
- moved C15 47.5 mm to (414.0, 124.4)
- moved C26 47.5 mm to (422.2, 124.4)
- moved C13 47.5 mm to (414.0, 116.3)
- moved C14 47.5 mm to (414.0, 120.4)
- moved C20 46.2 mm to (422.2, 112.3)
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Connections:
- C12 pad 1: Net-(A1-3V3) -> Net-(U3-S8)
- C13 pad 1: M1_A2 -> M1_3.3V
- C14 pad 1: M1_A3 -> M1_3.3V
- C16 pad 1: M2_3.3V -> Net-(A1-3V3)
- C17 pad 1: M2_NON_IN_1 -> M1_A2
- C18 pad 1: M2_3.3V -> M1_A3
- C19 pad 1: M2_3.3V -> M1_3.3V
- C20 pad 1: M2_NON_IN_2 -> M2_3.3V
- C21 pad 1: Net-(U11-S8) -> M2_NON_IN_1
- C24 pad 1: M2_3.3V -> M2_NON_IN_2
- C25 pad 1: Net-(A2-3V3) -> Net-(U11-S8)
- C26 pad 1: M2_A2 -> M2_3.3V
- C27 pad 1: M2_A3 -> M2_3.3V
- C9 pad 1: M1_3.3V -> M1_NON_IN_2
- R15 pad 2: Net-(U5-D) -> Net-(U3-D)
- R17 pad 1: Net-(U5-D) -> Net-(U3-D)
- R5 pad 1: Net-(J1-CC1) -> M1_NON_IN_1
- R5 pad 2: GND -> Net-(U2-D)
- R6 pad 1: M1_NON_IN_1 -> Net-(J1-CC1)
- R6 pad 2: Net-(U2-D) -> GND
- TP12 pad 1: Net-(J4-Pin_4) -> GND
- TP13 pad 1: Net-(J4-Pin_2) -> M1_A2
- TP14 pad 1: GND -> M1_A3
- TP15 pad 1: M1_A2 -> M1_3.3V
- TP16 pad 1: M1_A3 -> M1_A2
- TP17 pad 1: M1_3.3V -> M1_A3
- TP18 pad 1: M1_A2 -> Net-(J4-Pin_4)
- TP19 pad 1: M1_A3 -> Net-(J4-Pin_2)
- TP3 pad 1: +5V -> M1_GPIO_19
- TP4 pad 1: M1_GPIO_19 -> +5V
- TP8 pad 1: Net-(U5-S8) -> Net-(U3-S8)
- U3 pad 1: +5V -> M1_GPIO_14
- U3 pad 2: GND -> M1_GPIO_27
- U3 pad 4: unconnected-(U3-NC-Pad4) -> M1_ROW_9
- U3 pad 5: GND -> M1_ROW_10
- U3 pad 6: M1_VBUS -> M1_ROW_11
- U4 pad 1: +5V -> M1_COL_26
- U4 pad 2: GND -> M1_COL_25
- U4 pad 3: GND -> M1_COL_24
- U4 pad 4: unconnected-(U4-NC-Pad4) -> M1_COL_23
- U4 pad 5: GND -> M1_COL_22
- U4 pad 6: M2_VBUS -> M1_COL_21
- U5 pad 1: M1_GPIO_14 -> +5V
- U5 pad 2: M1_GPIO_27 -> GND
- U5 pad 4: M1_ROW_9 -> unconnected-(U5-NC-Pad4)
- U5 pad 5: M1_ROW_10 -> GND
- U5 pad 6: M1_ROW_11 -> M1_VBUS
- U6 pad 1: M1_COL_26 -> +5V
- U6 pad 2: M1_COL_25 -> GND
- U6 pad 3: M1_COL_24 -> GND
- U6 pad 4: M1_COL_23 -> unconnected-(U6-NC-Pad4)
- U6 pad 5: M1_COL_22 -> GND
- U6 pad 6: M1_COL_21 -> M2_VBUS
- U7 pad 2: Net-(U5-S8) -> Net-(U3-S8)
Other:
- copper layers 2 -> 4
