File: Finalized Logic Schematic/inventeam_final_schematic/inventeam_final_schematic.kicad_pcb (KiCad board)
At the start: 4 copper layers, 135 parts, among them J1 USB_C_Receptacle_PowerOnly_6P, J2 Conn_01x02, J3 Conn_02x20_Odd_Even, J4 Screw_Terminal_01x04, J5 JST Female, J6 JST Male, J7 JST Female, J8 JST Male, J9 Conn_02x20_Odd_Even, U1 MCP23S17_SP, U10 TMUX1208PW, U11 TMUX1208PW, U12 MCP23S17_SP, U13 MCP1525-TO, U14 OPA2333xxD, U2 TMUX1208PW, U3 TMUX1208PW, U4 MCP23S17_SP, U5 LM66100DCK, U6 LM66100DCK, U7 MCP1525-TO, U8 OPA2333xxD, U9 MCP23S17_SP

Commit message: Removed extra 0.1uf capacitor
Parts:
- removed A1, A2: Adafruit_Feather_HUZZAH32_ESP32, Module:Adafruit_Feather
- removed C1, C13, C14, C15, C17, C18, C19, C20, C22, C23, C26, C27, C28, C3, C30, C31, C32, C5, C6: 0.1uf, Capacitor_THT:C_Disc_D5.0mm_W2.5mm_P5.00mm
- removed C12, C16, C25, C29: 10uf, Capacitor_THT:C_Disc_D5.0mm_W2.5mm_P2.50mm
- removed C2, C21, C24, C9: 1nf, Capacitor_THT:CP_Axial_L10.0mm_D4.5mm_P15.00mm_Horizontal
- removed C4: 47uf, Capacitor_THT:CP_Radial_D5.0mm_P2.50mm
- removed D1: 1.5KE6.8A, Diode_THT:D_DO-201_P15.24mm_Horizontal
- removed D2, D3: SMF3.3A, Diode_SMD:D_SOD-123F
- removed F1, F2, F3: 1A, X16_GF100_PPTC:X16 GF100
- removed H1, H2, H3, H4: Mounting Hole, MountingHole:MountingHole_2.5mm_Pad
- removed J1: USB_C_Receptacle_PowerOnly_6P, Connector_USB:USB_C_Receptacle_GCT_USB4125-xx-x_6P_TopMnt_Horizontal
- removed J2: Conn_01x02, Connector_PinHeader_2.54mm:PinHeader_1x02_P2.54mm_Vertical
- removed J3, J9: Conn_02x20_Odd_Even, Connector_PinHeader_2.54mm:PinHeader_2x20_P2.54mm_Vertical
- removed J4: Screw_Terminal_01x04, TerminalBlock:TerminalBlock_Xinya_XY308-2.54-4P_1x04_P2.54mm_Horizontal
- removed J5, J7: JST Female, Connector_PinHeader_2.54mm:PinHeader_1x02_P2.54mm_Vertical
- removed J6, J8: JST Male, Connector_PinHeader_2.54mm:PinHeader_1x02_P2.54mm_Vertical
- removed R1, R10, R11, R12, R13, R14, R16, R18, R2, R21, R22, R23, R25, R26, R28, R29, R3, R30, R31, R32, R34, R36, R7, R8: 10k, Resistor_THT:R_Axial_DIN0207_L6.3mm_D2.5mm_P7.62mm_Horizontal
- removed R15, R24, R33, R5: 220, Resistor_THT:R_Axial_DIN0207_L6.3mm_D2.5mm_P10.16mm_Horizontal
- removed R17, R27, R35, R9: 1M, Resistor_THT:R_Axial_DIN0207_L6.3mm_D2.5mm_P7.62mm_Horizontal
- removed R19, R20, R37, R38: 1k, Resistor_THT:R_Axial_DIN0207_L6.3mm_D2.5mm_P7.62mm_Horizontal
- removed R4, R6: 5.1k, Resistor_THT:R_Axial_DIN0207_L6.3mm_D2.5mm_P7.62mm_Horizontal
- removed TP1, TP10, TP11, TP12, TP13, TP14, TP15, TP16, TP17, TP18, TP19, TP2, TP20, TP21, TP22, TP23, TP24, TP25, TP26, TP27, TP28, TP29, TP3, TP30, TP31, TP32, TP33, TP34, TP4, TP5, TP6, TP7, TP8, TP9: TestPoint_Probe, TestPoint:TestPoint_Pad_D1.0mm
- removed U1, U12, U4, U9: MCP23S17_SP, Package_DIP:DIP-28_W7.62mm
- removed U10, U11, U2, U3: TMUX1208PW, Package_SO:TSSOP-16_4.4x5mm_P0.65mm
- removed U13, U7: MCP1525-TO, Package_TO_SOT_THT:TO-92_Inline
- removed U14, U8: OPA2333xxD, Package_SO:SOIC-8_3.9x4.9mm_P1.27mm
- removed U5, U6: LM66100DCK, Package_TO_SOT_SMD:SOT-363_SC-70-6

Commit message: Work on PCB for logic schematic
Parts:
- added A1: Adafruit_Feather_HUZZAH32_ESP32, Module:Adafruit_Feather, F.Cu at (629.3, 81.6)
- added A2: Adafruit_Feather_HUZZAH32_ESP32, Module:Adafruit_Feather, F.Cu at (689.3, 81.6)
- added C1: 0.1uf, Capacitor_THT:C_Disc_D5.0mm_W2.5mm_P5.00mm, F.Cu at (395.3, 114.9)
- added C10: 1uf, Capacitor_THT:CP_Axial_L10.0mm_D4.5mm_P15.00mm_Horizontal, F.Cu at (594.0, 83.8)
- added C11: 10uf, Capacitor_THT:C_Disc_D5.0mm_W2.5mm_P2.50mm, F.Cu at (423.4, 91.9)
- added C12: 0.1uf, Capacitor_THT:C_Disc_D5.0mm_W2.5mm_P5.00mm, F.Cu at (395.3, 135.1)
- added C13: 0.1uf, Capacitor_THT:C_Disc_D5.0mm_W2.5mm_P5.00mm, F.Cu at (395.3, 139.2)
- added C14: 0.1uf, Capacitor_THT:C_Disc_D5.0mm_W2.5mm_P5.00mm, F.Cu at (403.5, 114.9)
- added C15: 10uf, Capacitor_THT:C_Disc_D5.0mm_W2.5mm_P2.50mm, F.Cu at (623.9, 84.2)
- added C16: 0.1uf, Capacitor_THT:C_Disc_D5.0mm_W2.5mm_P5.00mm, F.Cu at (403.5, 118.9)
- added C17: 0.1uf, Capacitor_THT:C_Disc_D5.0mm_W2.5mm_P5.00mm, F.Cu at (403.5, 123.0)
- added C18: 0.1uf, Capacitor_THT:C_Disc_D5.0mm_W2.5mm_P5.00mm, F.Cu at (620.7, 92.1)
- added C19: 0.1uf, Capacitor_THT:C_Disc_D5.0mm_W2.5mm_P5.00mm, F.Cu at (403.5, 131.1)
- added C2: 1nf, Capacitor_THT:CP_Axial_L10.0mm_D4.5mm_P15.00mm_Horizontal, F.Cu at (395.5, 77.2)
- added C20: 1nf, Capacitor_THT:CP_Axial_L10.0mm_D4.5mm_P15.00mm_Horizontal, F.Cu at (395.5, 103.3)
- added C21: 0.1uf, Capacitor_THT:C_Disc_D5.0mm_W2.5mm_P5.00mm, F.Cu at (403.5, 135.1)
- added C22: 0.1uf, Capacitor_THT:C_Disc_D5.0mm_W2.5mm_P5.00mm, F.Cu at (403.5, 139.2)
- added C23: 1nf, Capacitor_THT:CP_Axial_L10.0mm_D4.5mm_P15.00mm_Horizontal, F.Cu at (395.5, 109.8)
- added C24: 10uf, Capacitor_THT:C_Disc_D5.0mm_W2.5mm_P2.50mm, F.Cu at (423.4, 100.0)
- added C25: 0.1uf, Capacitor_THT:C_Disc_D5.0mm_W2.5mm_P5.00mm, F.Cu at (411.6, 114.9)
- added C26: 0.1uf, Capacitor_THT:C_Disc_D5.0mm_W2.5mm_P5.00mm, F.Cu at (411.6, 118.9)
- added C27: 0.1uf, Capacitor_THT:C_Disc_D5.0mm_W2.5mm_P5.00mm, F.Cu at (411.6, 123.0)
- added C28: 10uf, Capacitor_THT:C_Disc_D5.0mm_W2.5mm_P2.50mm, F.Cu at (683.9, 84.2)
- added C29: 0.1uf, Capacitor_THT:C_Disc_D5.0mm_W2.5mm_P5.00mm, F.Cu at (411.6, 127.0)
- added C3: 47uf, Capacitor_THT:CP_Radial_D5.0mm_P2.50mm, F.Cu at (577.3, 87.1)
- added C30: 0.1uf, Capacitor_THT:C_Disc_D5.0mm_W2.5mm_P5.00mm, F.Cu at (411.6, 131.1)
- added C31: 0.1uf, Capacitor_THT:C_Disc_D5.0mm_W2.5mm_P5.00mm, F.Cu at (680.7, 92.1)
- added C4: 0.1uf, Capacitor_THT:C_Disc_D5.0mm_W2.5mm_P5.00mm, F.Cu at (395.3, 118.9)
- added C5: 0.1uf, Capacitor_THT:C_Disc_D5.0mm_W2.5mm_P5.00mm, F.Cu at (395.3, 123.0)
- added C6: 0.1uf, Capacitor_THT:C_Disc_D5.0mm_W2.5mm_P5.00mm, F.Cu at (589.1, 83.8)
- added C7: 0.1uf, Capacitor_THT:C_Disc_D5.0mm_W2.5mm_P5.00mm, F.Cu at (589.8, 102.8)
- added C8: 1nf, Capacitor_THT:CP_Axial_L10.0mm_D4.5mm_P15.00mm_Horizontal, F.Cu at (395.5, 83.7)
- added C9: 1uf, Capacitor_THT:CP_Axial_L10.0mm_D4.5mm_P15.00mm_Horizontal, F.Cu at (594.0, 102.8)
- added D1: 1.5KE6.8A, Diode_THT:D_DO-201_P15.24mm_Horizontal, F.Cu at (584.2, 98.3)
- added D2: SMF3.3A, Diode_SMD:D_SOD-123F, F.Cu at (622.1, 95.0)
- added D3: SMF3.3A, Diode_SMD:D_SOD-123F, F.Cu at (682.1, 95.0)
- added F1: 1A, X16_GF100_PPTC:X16 GF100, F.Cu at (578.7, 98.4)
- added F2: 1A, X16_GF100_PPTC:X16 GF100, F.Cu at (620.6, 84.2)
- added F3: 1A, X16_GF100_PPTC:X16 GF100, F.Cu at (680.6, 84.2)
- added H1: Mounting Hole, MountingHole:MountingHole_2.5mm_Pad, F.Cu at (425.8, 40.5)
- added H2: Mounting Hole, MountingHole:MountingHole_2.5mm_Pad, F.Cu at (425.8, 47.0)
- added H3: Mounting Hole, MountingHole:MountingHole_2.5mm_Pad, F.Cu at (425.8, 53.6)
- added H4: Mounting Hole, MountingHole:MountingHole_2.5mm_Pad, F.Cu at (425.8, 60.1)
- added J1: USB_C_Receptacle_PowerOnly_6P, Connector_USB:USB_C_Receptacle_GCT_USB4125-xx-x_6P_TopMnt_Horizontal, F.Cu at (587.5, 73.0)
- added J2: Conn_01x02, Connector_PinHeader_2.54mm:PinHeader_1x02_P2.54mm_Vertical, F.Cu at (577.2, 81.4)
- added J3: Conn_02x20_Odd_Even, Connector_PinHeader_2.54mm:PinHeader_2x20_P2.54mm_Vertical, F.Cu at (381.7, 76.0)
- added J4: Screw_Terminal_01x04, TerminalBlock:TerminalBlock_Xinya_XY308-2.54-4P_1x04_P2.54mm_Horizontal, F.Cu at (731.2, 103.7)
- added J5: JST Female, Connector_PinHeader_2.54mm:PinHeader_1x02_P2.54mm_Vertical, F.Cu at (731.2, 109.2)
- added J6: JST Male, Connector_PinHeader_2.54mm:PinHeader_1x02_P2.54mm_Vertical, F.Cu at (722.3, 84.5)
- added J7: JST Female, Connector_PinHeader_2.54mm:PinHeader_1x02_P2.54mm_Vertical, F.Cu at (731.2, 117.9)
- added J8: JST Male, Connector_PinHeader_2.54mm:PinHeader_1x02_P2.54mm_Vertical, F.Cu at (662.3, 84.5)
- added J9: Conn_02x20_Odd_Even, Connector_PinHeader_2.54mm:PinHeader_2x20_P2.54mm_Vertical, F.Cu at (388.9, 76.0)
- added R1: 10k, Resistor_THT:R_Axial_DIN0207_L6.3mm_D2.5mm_P7.62mm_Horizontal, F.Cu at (591.0, 26.6)
- added R10: 10k, Resistor_THT:R_Axial_DIN0207_L6.3mm_D2.5mm_P7.62mm_Horizontal, F.Cu at (566.0, 26.6)
- added R11: 10k, Resistor_THT:R_Axial_DIN0207_L6.3mm_D2.5mm_P7.62mm_Horizontal, F.Cu at (561.0, 26.6)
- added R12: 10k, Resistor_THT:R_Axial_DIN0207_L6.3mm_D2.5mm_P7.62mm_Horizontal, F.Cu at (556.0, 26.6)
- added R13: 10k, Resistor_THT:R_Axial_DIN0207_L6.3mm_D2.5mm_P7.62mm_Horizontal, F.Cu at (551.0, 26.6)
- added R14: 10k, Resistor_THT:R_Axial_DIN0207_L6.3mm_D2.5mm_P7.62mm_Horizontal, F.Cu at (546.0, 26.6)
- added R15: 220, Resistor_THT:R_Axial_DIN0207_L6.3mm_D2.5mm_P10.16mm_Horizontal, F.Cu at (423.0, 79.7)
- added R16: 10k, Resistor_THT:R_Axial_DIN0207_L6.3mm_D2.5mm_P7.62mm_Horizontal, F.Cu at (541.0, 26.6)
- added R17: 1M, Resistor_THT:R_Axial_DIN0207_L6.3mm_D2.5mm_P7.62mm_Horizontal, F.Cu at (391.8, 59.5)
- added R18: 10k, Resistor_THT:R_Axial_DIN0207_L6.3mm_D2.5mm_P7.62mm_Horizontal, F.Cu at (536.0, 26.6)
- added R19: 1k, Resistor_THT:R_Axial_DIN0207_L6.3mm_D2.5mm_P7.62mm_Horizontal, F.Cu at (391.8, 67.6)
- added R2: 10k, Resistor_THT:R_Axial_DIN0207_L6.3mm_D2.5mm_P7.62mm_Horizontal, F.Cu at (586.0, 26.6)
- added R20: 1k, Resistor_THT:R_Axial_DIN0207_L6.3mm_D2.5mm_P7.62mm_Horizontal, F.Cu at (391.8, 71.6)
- added R21: 10k, Resistor_THT:R_Axial_DIN0207_L6.3mm_D2.5mm_P7.62mm_Horizontal, F.Cu at (673.4, 29.4)
- added R22: 10k, Resistor_THT:R_Axial_DIN0207_L6.3mm_D2.5mm_P7.62mm_Horizontal, F.Cu at (668.4, 29.4)
- added R23: 10k, Resistor_THT:R_Axial_DIN0207_L6.3mm_D2.5mm_P7.62mm_Horizontal, F.Cu at (663.4, 29.4)
- added R24: 220, Resistor_THT:R_Axial_DIN0207_L6.3mm_D2.5mm_P10.16mm_Horizontal, F.Cu at (423.0, 83.8)
- added R25: 10k, Resistor_THT:R_Axial_DIN0207_L6.3mm_D2.5mm_P7.62mm_Horizontal, F.Cu at (658.4, 29.4)
- added R26: 10k, Resistor_THT:R_Axial_DIN0207_L6.3mm_D2.5mm_P7.62mm_Horizontal, F.Cu at (653.4, 29.4)
- added R27: 1M, Resistor_THT:R_Axial_DIN0207_L6.3mm_D2.5mm_P7.62mm_Horizontal, F.Cu at (402.6, 59.5)
- added R28: 10k, Resistor_THT:R_Axial_DIN0207_L6.3mm_D2.5mm_P7.62mm_Horizontal, F.Cu at (648.4, 29.4)
- added R29: 10k, Resistor_THT:R_Axial_DIN0207_L6.3mm_D2.5mm_P7.62mm_Horizontal, F.Cu at (643.4, 29.4)
- added R3: 10k, Resistor_THT:R_Axial_DIN0207_L6.3mm_D2.5mm_P7.62mm_Horizontal, F.Cu at (581.0, 26.6)
- added R30: 10k, Resistor_THT:R_Axial_DIN0207_L6.3mm_D2.5mm_P7.62mm_Horizontal, F.Cu at (638.4, 29.4)
- added R31: 10k, Resistor_THT:R_Axial_DIN0207_L6.3mm_D2.5mm_P7.62mm_Horizontal, F.Cu at (633.4, 29.4)
- added R32: 10k, Resistor_THT:R_Axial_DIN0207_L6.3mm_D2.5mm_P7.62mm_Horizontal, F.Cu at (628.4, 29.4)
- added R33: 220, Resistor_THT:R_Axial_DIN0207_L6.3mm_D2.5mm_P10.16mm_Horizontal, F.Cu at (423.0, 87.8)
- added R34: 10k, Resistor_THT:R_Axial_DIN0207_L6.3mm_D2.5mm_P7.62mm_Horizontal, F.Cu at (623.4, 29.4)
- added R35: 1M, Resistor_THT:R_Axial_DIN0207_L6.3mm_D2.5mm_P7.62mm_Horizontal, F.Cu at (413.3, 51.4)
- added R36: 10k, Resistor_THT:R_Axial_DIN0207_L6.3mm_D2.5mm_P7.62mm_Horizontal, F.Cu at (618.4, 29.4)
- added R37: 1k, Resistor_THT:R_Axial_DIN0207_L6.3mm_D2.5mm_P7.62mm_Horizontal, F.Cu at (413.3, 59.5)
- added R38: 1k, Resistor_THT:R_Axial_DIN0207_L6.3mm_D2.5mm_P7.62mm_Horizontal, F.Cu at (413.3, 63.5)
- added R4: 5.1k, Resistor_THT:R_Axial_DIN0207_L6.3mm_D2.5mm_P7.62mm_Horizontal, F.Cu at (595.3, 79.6)
- added R5: 220, Resistor_THT:R_Axial_DIN0207_L6.3mm_D2.5mm_P10.16mm_Horizontal, F.Cu at (423.0, 75.7)
- added R6: 5.1k, Resistor_THT:R_Axial_DIN0207_L6.3mm_D2.5mm_P7.62mm_Horizontal, F.Cu at (595.3, 74.8)
- added R7: 10k, Resistor_THT:R_Axial_DIN0207_L6.3mm_D2.5mm_P7.62mm_Horizontal, F.Cu at (576.0, 26.6)
- added R8: 10k, Resistor_THT:R_Axial_DIN0207_L6.3mm_D2.5mm_P7.62mm_Horizontal, F.Cu at (571.0, 26.6)
- added R9: 1M, Resistor_THT:R_Axial_DIN0207_L6.3mm_D2.5mm_P7.62mm_Horizontal, F.Cu at (380.1, 66.8)
- added TP1: TestPoint_Probe, TestPoint:TestPoint_Pad_D1.0mm, F.Cu at (600.8, 119.5)
- added TP10: TestPoint_Probe, TestPoint:TestPoint_Pad_D1.0mm, F.Cu at (422.8, 120.5)
- added TP11: TestPoint_Probe, TestPoint:TestPoint_Pad_D1.0mm, F.Cu at (422.8, 123.5)
- added TP12: TestPoint_Probe, TestPoint:TestPoint_Pad_D1.0mm, F.Cu at (613.2, 89.7)
- added TP13: TestPoint_Probe, TestPoint:TestPoint_Pad_D1.0mm, F.Cu at (422.8, 129.6)
- added TP14: TestPoint_Probe, TestPoint:TestPoint_Pad_D1.0mm, F.Cu at (422.8, 132.7)
- added TP15: TestPoint_Probe, TestPoint:TestPoint_Pad_D1.0mm, F.Cu at (616.8, 100.0)
- added TP16: TestPoint_Probe, TestPoint:TestPoint_Pad_D1.0mm, F.Cu at (425.8, 117.4)
- added TP17: TestPoint_Probe, TestPoint:TestPoint_Pad_D1.0mm, F.Cu at (425.8, 120.5)
- added TP18: TestPoint_Probe, TestPoint:TestPoint_Pad_D1.0mm, F.Cu at (425.8, 123.5)
- added TP19: TestPoint_Probe, TestPoint:TestPoint_Pad_D1.0mm, F.Cu at (425.8, 126.6)
- added TP2: TestPoint_Probe, TestPoint:TestPoint_Pad_D1.0mm, F.Cu at (419.7, 117.4)
- added TP20: TestPoint_Probe, TestPoint:TestPoint_Pad_D1.0mm, F.Cu at (425.8, 129.6)
- added TP21: TestPoint_Probe, TestPoint:TestPoint_Pad_D1.0mm, F.Cu at (425.8, 132.7)
- added TP22: TestPoint_Probe, TestPoint:TestPoint_Pad_D1.0mm, F.Cu at (428.9, 114.4)
- added TP23: TestPoint_Probe, TestPoint:TestPoint_Pad_D1.0mm, F.Cu at (428.9, 117.4)
- added TP24: TestPoint_Probe, TestPoint:TestPoint_Pad_D1.0mm, F.Cu at (428.9, 120.5)
- added TP25: TestPoint_Probe, TestPoint:TestPoint_Pad_D1.0mm, F.Cu at (428.9, 123.5)
- added TP26: TestPoint_Probe, TestPoint:TestPoint_Pad_D1.0mm, F.Cu at (428.9, 126.6)
- added TP27: TestPoint_Probe, TestPoint:TestPoint_Pad_D1.0mm, F.Cu at (428.9, 129.6)
- added TP28: TestPoint_Probe, TestPoint:TestPoint_Pad_D1.0mm, F.Cu at (428.9, 132.7)
- added TP29: TestPoint_Probe, TestPoint:TestPoint_Pad_D1.0mm, F.Cu at (673.2, 89.7)
- added TP3: TestPoint_Probe, TestPoint:TestPoint_Pad_D1.0mm, F.Cu at (419.7, 120.5)
- added TP30: TestPoint_Probe, TestPoint:TestPoint_Pad_D1.0mm, F.Cu at (431.9, 117.4)
- added TP31: TestPoint_Probe, TestPoint:TestPoint_Pad_D1.0mm, F.Cu at (431.9, 120.5)
- added TP32: TestPoint_Probe, TestPoint:TestPoint_Pad_D1.0mm, F.Cu at (676.8, 100.0)
- added TP33: TestPoint_Probe, TestPoint:TestPoint_Pad_D1.0mm, F.Cu at (431.9, 126.6)
- added TP34: TestPoint_Probe, TestPoint:TestPoint_Pad_D1.0mm, F.Cu at (431.9, 129.6)
- added TP4: TestPoint_Probe, TestPoint:TestPoint_Pad_D1.0mm, F.Cu at (575.7, 109.1)
- added TP5: TestPoint_Probe, TestPoint:TestPoint_Pad_D1.0mm, F.Cu at (419.7, 126.6)
- added TP6: TestPoint_Probe, TestPoint:TestPoint_Pad_D1.0mm, F.Cu at (419.7, 129.6)
- added TP7: TestPoint_Probe, TestPoint:TestPoint_Pad_D1.0mm, F.Cu at (419.7, 132.7)
- added TP8: TestPoint_Probe, TestPoint:TestPoint_Pad_D1.0mm, F.Cu at (422.8, 114.4)
- added TP9: TestPoint_Probe, TestPoint:TestPoint_Pad_D1.0mm, F.Cu at (422.8, 117.4)
- added U1: MCP23S17_SP, Package_DIP:DIP-28_W7.62mm, F.Cu at (331.8, 91.6)
- added U10: TMUX1208PW, Package_SO:TSSOP-16_4.4x5mm_P0.65mm, F.Cu at (417.0, 90.1)
- added U11: TMUX1208PW, Package_SO:TSSOP-16_4.4x5mm_P0.65mm, F.Cu at (417.0, 96.7)
- added U12: MCP23S17_SP, Package_DIP:DIP-28_W7.62mm, F.Cu at (364.1, 91.6)
- added U13: MCP1525-TO, Package_TO_SOT_THT:TO-92_Inline, F.Cu at (429.9, 98.9)
- added U14: OPA2333xxD, Package_SO:SOIC-8_3.9x4.9mm_P1.27mm, F.Cu at (370.1, 136.6)
- added U2: TMUX1208PW, Package_SO:TSSOP-16_4.4x5mm_P0.65mm, F.Cu at (417.0, 77.0)
- added U3: TMUX1208PW, Package_SO:TSSOP-16_4.4x5mm_P0.65mm, F.Cu at (417.0, 83.5)
- added U4: MCP23S17_SP, Package_DIP:DIP-28_W7.62mm, F.Cu at (342.6, 91.6)
- added U5: LM66100DCK, Package_TO_SOT_SMD:SOT-363_SC-70-6, F.Cu at (598.4, 82.9)
- added U6: LM66100DCK, Package_TO_SOT_SMD:SOT-363_SC-70-6, F.Cu at (598.5, 102.0)
- added U7: MCP1525-TO, Package_TO_SOT_THT:TO-92_Inline, F.Cu at (429.9, 93.1)
- added U8: OPA2333xxD, Package_SO:SOIC-8_3.9x4.9mm_P1.27mm, F.Cu at (370.1, 130.0)
- added U9: MCP23S17_SP, Package_DIP:DIP-28_W7.62mm, F.Cu at (353.3, 91.6)
- added kibuzzard-69C8846F: G***, kibuzzard-69C8846F, F.Cu at (584.0, 123.9)
- added kibuzzard-69C8AE86: G***, kibuzzard-69C8AE86, F.Cu at (669.8, 125.7)
Routing:
- net M2_VBUS: track 0.00 -> 151.1 mm
- net Net-(J4-Pin_1): track 0.00 -> 108.3 mm
- net M1_TX: track 0.00 -> 104.7 mm
- net M2_TX: track 0.00 -> 100.5 mm
- net Net-(J7-Pin_2): track 0.00 -> 100.5 mm
- net M1_VBUS: track 0.00 -> 78.5 mm
- net +5V: track 0.00 -> 59.0 mm
- net Net-(J5-Pin_2): track 0.00 -> 31.6 mm
- net Net-(J2-Pin_1): track 0.00 -> 25.1 mm
- net Net-(J4-Pin_3): track 0.00 -> 22.0 mm
- net Net-(J4-Pin_2): track 0.00 -> 21.8 mm
- net Net-(J4-Pin_4): track 0.00 -> 16.6 mm
- net M2_3.3V: track 0.00 -> 14.0 mm
- net M1_3.3V: track 0.00 -> 14.0 mm
- net Net-(J1-CC2): track 0.00 -> 10.0 mm
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Other:
- board text added: "+BATT"
- board text added: "-BATT"
- board text added: "Mismatched battery-wiring is not protected!"
- board text added: "Never have more than one USB connection!"
- board text added: "Test +3.3V"
- board text added: "Test +5V"
- board text added: "Test GND"
