File: Finalized Logic Schematic/inventeam_final_schematic/inventeam_final_schematic.kicad_pcb (KiCad board)
At the start: 4 copper layers, 140 parts, among them J1 USB_C_Receptacle_PowerOnly_6P, J2 Conn_01x02, J3 Conn_02x20_Odd_Even, J4 Screw_Terminal_01x04, J5 JST Female, J6 JST Male, J7 JST Female, J8 JST Male, J9 Conn_02x20_Odd_Even, U1 MCP23S17_SP, U10 TMUX1208PW, U11 TMUX1208PW, U12 MCP23S17_SP, U13 MCP1525-TO, U14 OPA2333xxD, U2 TMUX1208PW, U3 TMUX1208PW, U4 MCP23S17_SP, U5 LM66100DCK, U6 LM66100DCK, U7 MCP1525-TO, U8 OPA2333xxD, U9 MCP23S17_SP

Commit message: Logic schematic V2
Parts:
- removed A1, A2: Adafruit_Feather_HUZZAH32_ESP32, Module:Adafruit_Feather
- removed C1, C12, C13, C14, C16, C17, C18, C19, C21, C22, C25, C26, C27, C29, C30, C31, C4, C5, C6, C7: 0.1uf, Capacitor_THT:C_Disc_D5.0mm_W2.5mm_P5.00mm
- removed C10, C9: 1uf, Capacitor_THT:CP_Axial_L10.0mm_D4.5mm_P15.00mm_Horizontal
- removed C11, C15, C24, C28: 10uf, Capacitor_THT:C_Disc_D5.0mm_W2.5mm_P2.50mm
- removed C2, C20, C23, C8: 1nf, Capacitor_THT:CP_Axial_L10.0mm_D4.5mm_P15.00mm_Horizontal
- removed C3: 47uf, Capacitor_THT:CP_Radial_D5.0mm_P2.50mm
- removed D1: 1.5KE6.8A, Diode_THT:D_DO-201_P15.24mm_Horizontal
- removed D2, D3: SMF3.3A, Diode_SMD:D_SOD-123F
- removed F1, F2, F3: 1A, X16_GF100_PPTC:X16 GF100
- removed H1, H2, H3, H4: Mounting Hole, MountingHole:MountingHole_2.5mm_Pad
- removed J1: USB_C_Receptacle_PowerOnly_6P, Connector_USB:USB_C_Receptacle_GCT_USB4125-xx-x_6P_TopMnt_Horizontal
- removed J2: Conn_01x02, Connector_PinHeader_2.54mm:PinHeader_1x02_P2.54mm_Vertical
- removed J3, J9: Conn_02x20_Odd_Even, Connector_PinHeader_2.54mm:PinHeader_2x20_P2.54mm_Vertical
- removed J4: Screw_Terminal_01x04, TerminalBlock:TerminalBlock_Xinya_XY308-2.54-4P_1x04_P2.54mm_Horizontal
- removed J5, J7: JST Female, Connector_PinHeader_2.54mm:PinHeader_1x02_P2.54mm_Vertical
- removed J6, J8: JST Male, Connector_PinHeader_2.54mm:PinHeader_1x02_P2.54mm_Vertical
- removed R1, R10, R11, R12, R13, R14, R16, R18, R2, R21, R22, R23, R25, R26, R28, R29, R3, R30, R31, R32, R34, R36, R7, R8: 10k, Resistor_THT:R_Axial_DIN0207_L6.3mm_D2.5mm_P7.62mm_Horizontal
- removed R15, R24, R33, R5: 220, Resistor_THT:R_Axial_DIN0207_L6.3mm_D2.5mm_P10.16mm_Horizontal
- removed R17, R27, R35, R9: 1M, Resistor_THT:R_Axial_DIN0207_L6.3mm_D2.5mm_P7.62mm_Horizontal
- removed R19, R20, R37, R38: 1k, Resistor_THT:R_Axial_DIN0207_L6.3mm_D2.5mm_P7.62mm_Horizontal
- removed R4, R6: 5.1k, Resistor_THT:R_Axial_DIN0207_L6.3mm_D2.5mm_P7.62mm_Horizontal
- removed TP1, TP10, TP11, TP12, TP13, TP14, TP15, TP16, TP17, TP18, TP19, TP2, TP20, TP21, TP22, TP23, TP24, TP25, TP26, TP27, TP28, TP29, TP3, TP30, TP31, TP32, TP33, TP34, TP4, TP5, TP6, TP7, TP8, TP9: TestPoint_Probe, TestPoint:TestPoint_Pad_D1.0mm
- removed U1, U12, U4, U9: MCP23S17_SP, Package_DIP:DIP-28_W7.62mm
- removed U10, U11, U2, U3: TMUX1208PW, Package_SO:TSSOP-16_4.4x5mm_P0.65mm
- removed U13, U7: MCP1525-TO, Package_TO_SOT_THT:TO-92_Inline
- removed U14, U8: OPA2333xxD, Package_SO:SOIC-8_3.9x4.9mm_P1.27mm
- removed U5, U6: LM66100DCK, Package_TO_SOT_SMD:SOT-363_SC-70-6
- removed kibuzzard-69C8846F: G***, kibuzzard-69C8846F
- removed kibuzzard-69C8AE86: G***, kibuzzard-69C8AE86
Routing:
- net M2_VBUS: track 151.1 -> 0.00 mm
- net Net-(J4-Pin_1): track 108.3 -> 0.00 mm
- net M1_TX: track 104.7 -> 0.00 mm
- net M2_TX: track 100.5 -> 0.00 mm
- net Net-(J7-Pin_2): track 100.5 -> 0.00 mm
- net M1_VBUS: track 78.5 -> 0.00 mm
- net +5V: track 59.0 -> 0.00 mm
- net Net-(J5-Pin_2): track 31.6 -> 0.00 mm
- net Net-(J2-Pin_1): track 25.1 -> 0.00 mm
- net Net-(J4-Pin_3): track 22.0 -> 0.00 mm
- net Net-(J4-Pin_2): track 21.8 -> 0.00 mm
- net Net-(J4-Pin_4): track 16.6 -> 0.00 mm
- net M2_3.3V: track 14.0 -> 0.00 mm
- net M1_3.3V: track 14.0 -> 0.00 mm
- net Net-(J1-CC2): track 10.0 -> 0.00 mm
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Other:
- board text removed: "+BATT"
- board text removed: "-BATT"
- board text removed: "Mismatched battery-wiring is not protected!"
- board text removed: "Never have more than one USB connection!"
- board text removed: "Test +3.3V"
- board text removed: "Test +5V"
- board text removed: "Test GND"
