File: Finalized Thermistor Schematic/inventeam_thermistor_schematic/inventeam_thermistor_schematic.kicad_sch (KiCad schematic)
At the start: 133 parts, among them J1 Header, J2 USB_C_Receptacle_PowerOnly_6P, J3 Screw_Terminal_01x04, J4 JST Female, J5 JST Male, J6 Header, J8 JST Female, J9 JST Male, U1 MCP23S17_SP, U10 TMUX1208PW, U11 TMUX1208PW, U12 MCP23S17_SP, U13 MCP1525-TO, U14 OPA2333xxD, U2 TMUX1208PW, U3 TMUX1208PW, U4 MCP23S17_SP, U5 LM66100DCK, U6 LM66100DCK, U7 MCP1525-TO, U8 OPA2333xxD, U9 MCP23S17_SP

Commit message: Ground header pin for thermistor pcb
Parts:
- removed A1, A2: Adafruit_Feather_HUZZAH32_ESP32, Module:Adafruit_Feather, symbol MCU_Module:Adafruit_Feather_HUZZAH32_ESP32
- removed C1, C10, C12, C13, C14, C15, C17, C18, C21, C22, C23, C25, C26, C27, C3, C4, C8, C9: 0.1uf, Capacitor_THT:CP_Radial_D5.0mm_P2.50mm, symbol Device:C_US
- removed C11, C20, C24, C7: 10uf, Capacitor_THT:CP_Radial_D5.0mm_P2.50mm, symbol Device:C_US
- removed C16, C19, C2, C5: 1nf, Capacitor_THT:CP_Axial_L10.0mm_D4.5mm_P15.00mm_Horizontal, symbol Device:C_US
- removed C6: 47uf, symbol Device:C_US
- removed D1: 1.5KE6.8A, Diode_THT:D_DO-201_P15.24mm_Horizontal, symbol Device:D_TVS
- removed D2, D3: SMF3.3A, Diode_SMD:D_SOD-123F, symbol Device:D_TVS
- removed F1: 2A, symbol Device:Polyfuse
- removed F2, F3: 1A, symbol Device:Polyfuse
- removed H1, H2, H3, H4: Mounting Hole, MountingHole:MountingHole_2.5mm_Pad, symbol Mechanical:MountingHole_Pad
- removed J2: USB_C_Receptacle_PowerOnly_6P, symbol Connector:USB_C_Receptacle_PowerOnly_6P
- removed J3: Screw_Terminal_01x04, TerminalBlock:TerminalBlock_Xinya_XY308-2.54-4P_1x04_P2.54mm_Horizontal, symbol Connector:Screw_Terminal_01x04
- removed J4, J8: JST Female, symbol Connector_Generic:Conn_01x02
- removed J5, J9: JST Male, symbol Connector_Generic:Conn_01x02
- removed J6: Header, symbol Connector_Generic:Conn_02x20_Top_Bottom
- removed R1, R10, R11, R12, R16, R18, R2, R21, R22, R23, R25, R26, R28, R29, R3, R30, R31, R32, R34, R36, R5, R6, R8, R9: 10k, Resistor_THT:R_Axial_DIN0207_L6.3mm_D2.5mm_P7.62mm_Horizontal, symbol Device:R_US
- removed R13, R24, R33, R4: 220, Resistor_THT:R_Axial_DIN0207_L6.3mm_D2.5mm_P10.16mm_Horizontal, symbol Device:R_US
- removed R14, R15: 5.1k, symbol Device:R_US
- removed R17, R27, R35, R7: 1M, Resistor_THT:R_Axial_DIN0207_L6.3mm_D2.5mm_P7.62mm_Horizontal, symbol Device:R_US
- removed R19, R20, R37, R38: 1k, Resistor_THT:R_Axial_DIN0207_L6.3mm_D2.5mm_P7.62mm_Horizontal, symbol Device:R_US
- removed TP1, TP10, TP11, TP12, TP13, TP14, TP15, TP16, TP17, TP18, TP19, TP2, TP20, TP21, TP22, TP23, TP24, TP25, TP26, TP27, TP28, TP29, TP3, TP30, TP31, TP32, TP33, TP34, TP4, TP5, TP6, TP7, TP8, TP9: TestPoint_Probe, TestPoint:TestPoint_Pad_D1.0mm, symbol Connector:TestPoint_Probe
- removed U1, U12, U4, U9: MCP23S17_SP, Package_DIP:DIP-28_W7.62mm, symbol Interface_Expansion:MCP23S17_SP
- removed U10, U11, U2, U3: TMUX1208PW, Package_SO:TSSOP-16_4.4x5mm_P0.65mm, symbol Analog_Switch:TMUX1208PW
- removed U13, U7: MCP1525-TO, Package_TO_SOT_THT:TO-92_Inline, symbol Reference_Voltage:MCP1525-TO
- removed U14, U8: OPA2333xxD, Package_SO:SOIC-8_3.9x4.9mm_P1.27mm, symbol Amplifier_Operational:OPA2333xxD
- removed U5, U6: LM66100DCK, Package_TO_SOT_SMD:SOT-363_SC-70-6, symbol Power_Management:LM66100DCK
- added TH1, TH10, TH100, TH101, TH102, TH103, TH104, TH105, TH106, TH107, TH108, TH109, TH11, TH110, TH111, TH112, TH113, TH114, TH115, TH116, TH117, TH118, TH119, TH12, TH120, TH121, TH122, TH123, TH124, TH125, TH126, TH127, TH128, TH129, TH13, TH130, TH131, TH132, TH133, TH134, TH135, TH136, TH137, TH138, TH139, TH14, TH140, TH141, TH142, TH143, TH144, TH145, TH146, TH147, TH148, TH149, TH15, TH150, TH151, TH152, TH153, TH154, TH155, TH156, TH157, TH158, TH159, TH16, TH160, TH161, TH162, TH163, TH164, TH165, TH166, TH167, TH168, TH169, TH17, TH170, TH171, TH172, TH173, TH174, TH175, TH176, TH177, TH178, TH179, TH18, TH180, TH181, TH182, TH183, TH184, TH185, TH186, TH187, TH188, TH189, TH19, TH190, TH191, TH192, TH193, TH194, TH195, TH196, TH197, TH198, TH199, TH2, TH20, TH200, TH201, TH202, TH203, TH204, TH205, TH206, TH207, TH208, TH209, TH21, TH210, TH211, TH212, TH213, TH214, TH215, TH216, TH217, TH218, TH219, TH22, TH220, TH221, TH222, TH223, TH224, TH225, TH226, TH227, TH228, TH229, TH23, TH230, TH231, TH232, TH233, TH234, TH235, TH236, TH237, TH238, TH239, TH24, TH240, TH241, TH242, TH243, TH244, TH245, TH246, TH247, TH248, TH249, TH25, TH250, TH251, TH252, TH253, TH254, TH255, TH256, TH257, TH258, TH259, TH26, TH260, TH261, TH262, TH263, TH264, TH265, TH266, TH267, TH268, TH269, TH27, TH270, TH271, TH272, TH273, TH274, TH275, TH276, TH277, TH278, TH279, TH28, TH280, TH281, TH282, TH283, TH284, TH285, TH286, TH287, TH288, TH289, TH29, TH290, TH291, TH292, TH293, TH294, TH295, TH296, TH297, TH298, TH299, TH3, TH30, TH300, TH301, TH302, TH303, TH304, TH305, TH306, TH307, TH308, TH309, TH31, TH310, TH311, TH312, TH32, TH33, TH34, TH35, TH36, TH37, TH38, TH39, TH4, TH40, TH41, TH42, TH43, TH44, TH45, TH46, TH47, TH48, TH49, TH5, TH50, TH51, TH52, TH53, TH54, TH55, TH56, TH57, TH58, TH59, TH6, TH60, TH61, TH62, TH63, TH64, TH65, TH66, TH67, TH68, TH69, TH7, TH70, TH71, TH72, TH73, TH74, TH75, TH76, TH77, TH78, TH79, TH8, TH80, TH81, TH82, TH83, TH84, TH85, TH86, TH87, TH88, TH89, TH9, TH90, TH91, TH92, TH93, TH94, TH95, TH96, TH97, TH98, TH99: 10k, symbol Device:Thermistor_NTC_US
Connections:
- net GND: no longer names the net of J1.32 (Pin_32)
- net M1_COL_1: no longer names the net of J1.5 (Pin_5)
- net M1_COL_10: no longer names the net of J1.23 (Pin_23)
- net M1_COL_11: no longer names the net of J1.22 (Pin_22)
- net M1_COL_12: no longer names the net of J1.21 (Pin_21)
- net M1_COL_13: no longer names the net of J1.4 (Pin_4)
- net M1_COL_14: no longer names the net of J1.3 (Pin_3)
- net M1_COL_15: no longer names the net of J1.2 (Pin_2)
- net M1_COL_16: no longer names the net of J1.1 (Pin_1)
- net M1_COL_17: no longer names the net of J1.16 (Pin_16)
- net M1_COL_18: no longer names the net of J1.15 (Pin_15)
- net M1_COL_19: no longer names the net of J1.14 (Pin_14)
- net M1_COL_2: no longer names the net of J1.6 (Pin_6)
- net M1_COL_20: no longer names the net of J1.13 (Pin_13)
- net M1_COL_21: no longer names the net of J1.30 (Pin_30)
- net M1_COL_22: no longer names the net of J1.29 (Pin_29)
- net M1_COL_23: no longer names the net of J1.9 (Pin_9)
- net M1_COL_24: no longer names the net of J1.10 (Pin_10)
- net M1_COL_25: no longer names the net of J1.11 (Pin_11)
- net M1_COL_26: no longer names the net of J1.12 (Pin_12)
- net M1_COL_3: no longer names the net of J1.7 (Pin_7)
- net M1_COL_4: no longer names the net of J1.8 (Pin_8)
- net M1_COL_5: no longer names the net of J1.25 (Pin_25)
- net M1_COL_6: no longer names the net of J1.26 (Pin_26)
- net M1_COL_7: no longer names the net of J1.27 (Pin_27)
- net M1_COL_8: no longer names the net of J1.28 (Pin_28)
- net M1_COL_9: no longer names the net of J1.24 (Pin_24)
- net M1_ROW_1: no longer names the net of J1.17 (Pin_17)
- net M1_ROW_10: no longer names the net of J1.35 (Pin_35)
- net M1_ROW_11: no longer names the net of J1.34 (Pin_34)
- net M1_ROW_12: no longer names the net of J1.33 (Pin_33)
- net M1_ROW_2: no longer names the net of J1.18 (Pin_18)
- net M1_ROW_3: no longer names the net of J1.19 (Pin_19)
- net M1_ROW_4: no longer names the net of J1.20 (Pin_20)
- net M1_ROW_5: no longer names the net of J1.40 (Pin_40)
- net M1_ROW_6: no longer names the net of J1.39 (Pin_39)
- net M1_ROW_7: no longer names the net of J1.38 (Pin_38)
- net M1_ROW_8: no longer names the net of J1.37 (Pin_37)
- net M1_ROW_9: no longer names the net of J1.36 (Pin_36)
- new net COL_1: TH1.1, TH10.1, TH11.1, TH12.1, TH2.1, TH3.1, TH4.1, TH5.1, TH6.1, TH7.1, TH8.1, TH9.1
- new net COL_10: TH109.1, TH110.1, TH111.1, TH112.1, TH113.1, TH114.1, TH115.1, TH116.1, TH117.1, TH118.1, TH119.1, TH120.1
- new net COL_11: TH121.1, TH122.1, TH123.1, TH124.1, TH125.1, TH126.1, TH127.1, TH128.1, TH129.1, TH130.1, TH131.1, TH132.1
- new net COL_12: TH133.1, TH134.1, TH135.1, TH136.1, TH137.1, TH138.1, TH139.1, TH140.1, TH141.1, TH142.1, TH143.1, TH144.1
- new net COL_13: TH145.1, TH146.1, TH147.1, TH148.1, TH149.1, TH150.1, TH151.1, TH152.1, TH153.1, TH154.1, TH155.1, TH156.1
- new net COL_14: TH157.1, TH158.1, TH159.1, TH160.1, TH161.1, TH162.1, TH163.1, TH164.1, TH165.1, TH166.1, TH167.1, TH168.1
- new net COL_15: TH169.1, TH170.1, TH171.1, TH172.1, TH173.1, TH174.1, TH175.1, TH176.1, TH177.1, TH178.1, TH179.1, TH180.1
- new net COL_16: TH181.1, TH182.1, TH183.1, TH184.1, TH185.1, TH186.1, TH187.1, TH188.1, TH189.1, TH190.1, TH191.1, TH192.1
- new net COL_17: TH193.1, TH194.1, TH195.1, TH196.1, TH197.1, TH198.1, TH199.1, TH200.1, TH201.1, TH202.1, TH203.1, TH204.1
- new net COL_18: TH205.1, TH206.1, TH207.1, TH208.1, TH209.1, TH210.1, TH211.1, TH212.1, TH213.1, TH214.1, TH215.1, TH216.1
- new net COL_19: TH217.1, TH218.1, TH219.1, TH220.1, TH221.1, TH222.1, TH223.1, TH224.1, TH225.1, TH226.1, TH227.1, TH228.1
- new net COL_2: TH13.1, TH14.1, TH15.1, TH16.1, TH17.1, TH18.1, TH19.1, TH20.1, TH21.1, TH22.1, TH23.1, TH24.1
- new net COL_20: TH229.1, TH230.1, TH231.1, TH232.1, TH233.1, TH234.1, TH235.1, TH236.1, TH237.1, TH238.1, TH239.1, TH240.1
- new net COL_21: TH241.1, TH242.1, TH243.1, TH244.1, TH245.1, TH246.1, TH247.1, TH248.1, TH249.1, TH250.1, TH251.1, TH252.1
- new net COL_22: TH253.1, TH254.1, TH255.1, TH256.1, TH257.1, TH258.1, TH259.1, TH260.1, TH261.1, TH262.1, TH263.1, TH264.1
- new net COL_23: TH265.1, TH266.1, TH267.1, TH268.1, TH269.1, TH270.1, TH271.1, TH272.1, TH273.1, TH274.1, TH275.1, TH276.1
- new net COL_24: TH277.1, TH278.1, TH279.1, TH280.1, TH281.1, TH282.1, TH283.1, TH284.1, TH285.1, TH286.1, TH287.1, TH288.1
- new net COL_25: TH289.1, TH290.1, TH291.1, TH292.1, TH293.1, TH294.1, TH295.1, TH296.1, TH297.1, TH298.1, TH299.1, TH300.1
- new net COL_26: TH301.1, TH302.1, TH303.1, TH304.1, TH305.1, TH306.1, TH307.1, TH308.1, TH309.1, TH310.1, TH311.1, TH312.1
- new net COL_3: TH25.1, TH26.1, TH27.1, TH28.1, TH29.1, TH30.1, TH31.1, TH32.1, TH33.1, TH34.1, TH35.1, TH36.1
- new net COL_4: TH37.1, TH38.1, TH39.1, TH40.1, TH41.1, TH42.1, TH43.1, TH44.1, TH45.1, TH46.1, TH47.1, TH48.1
- new net COL_5: TH49.1, TH50.1, TH51.1, TH52.1, TH53.1, TH54.1, TH55.1, TH56.1, TH57.1, TH58.1, TH59.1, TH60.1
- new net COL_6: TH61.1, TH62.1, TH63.1, TH64.1, TH65.1, TH66.1, TH67.1, TH68.1, TH69.1, TH70.1, TH71.1, TH72.1
- new net COL_7: TH73.1, TH74.1, TH75.1, TH76.1, TH77.1, TH78.1, TH79.1, TH80.1, TH81.1, TH82.1, TH83.1, TH84.1
- new net COL_8: TH85.1, TH86.1, TH87.1, TH88.1, TH89.1, TH90.1, TH91.1, TH92.1, TH93.1, TH94.1, TH95.1, TH96.1
- new net COL_9: TH100.1, TH101.1, TH102.1, TH103.1, TH104.1, TH105.1, TH106.1, TH107.1, TH108.1, TH97.1, TH98.1, TH99.1
- new net ROW_1: TH1.2, TH109.2, TH121.2, TH13.2, TH133.2, TH145.2, TH157.2, TH169.2, TH181.2, TH193.2, TH205.2, TH217.2, TH229.2, TH241.2, TH25.2, TH253.2, TH265.2, TH277.2, TH289.2, TH301.2, TH37.2, TH49.2, TH61.2, TH73.2, TH85.2, TH97.2
- new net ROW_10: TH10.2, TH106.2, TH118.2, TH130.2, TH142.2, TH154.2, TH166.2, TH178.2, TH190.2, TH202.2, TH214.2, TH22.2, TH226.2, TH238.2, TH250.2, TH262.2, TH274.2, TH286.2, TH298.2, TH310.2, TH34.2, TH46.2, TH58.2, TH70.2, TH82.2, TH94.2
- new net ROW_11: TH107.2, TH11.2, TH119.2, TH131.2, TH143.2, TH155.2, TH167.2, TH179.2, TH191.2, TH203.2, TH215.2, TH227.2, TH23.2, TH239.2, TH251.2, TH263.2, TH275.2, TH287.2, TH299.2, TH311.2, TH35.2, TH47.2, TH59.2, TH71.2, TH83.2, TH95.2
- new net ROW_12: TH108.2, TH12.2, TH120.2, TH132.2, TH144.2, TH156.2, TH168.2, TH180.2, TH192.2, TH204.2, TH216.2, TH228.2, TH24.2, TH240.2, TH252.2, TH264.2, TH276.2, TH288.2, TH300.2, TH312.2, TH36.2, TH48.2, TH60.2, TH72.2, TH84.2, TH96.2
- new net ROW_2: TH110.2, TH122.2, TH134.2, TH14.2, TH146.2, TH158.2, TH170.2, TH182.2, TH194.2, TH2.2, TH206.2, TH218.2, TH230.2, TH242.2, TH254.2, TH26.2, TH266.2, TH278.2, TH290.2, TH302.2, TH38.2, TH50.2, TH62.2, TH74.2, TH86.2, TH98.2
- new net ROW_3: TH111.2, TH123.2, TH135.2, TH147.2, TH15.2, TH159.2, TH171.2, TH183.2, TH195.2, TH207.2, TH219.2, TH231.2, TH243.2, TH255.2, TH267.2, TH27.2, TH279.2, TH291.2, TH3.2, TH303.2, TH39.2, TH51.2, TH63.2, TH75.2, TH87.2, TH99.2
- new net ROW_4: TH100.2, TH112.2, TH124.2, TH136.2, TH148.2, TH16.2, TH160.2, TH172.2, TH184.2, TH196.2, TH208.2, TH220.2, TH232.2, TH244.2, TH256.2, TH268.2, TH28.2, TH280.2, TH292.2, TH304.2, TH4.2, TH40.2, TH52.2, TH64.2, TH76.2, TH88.2
- new net ROW_5: TH101.2, TH113.2, TH125.2, TH137.2, TH149.2, TH161.2, TH17.2, TH173.2, TH185.2, TH197.2, TH209.2, TH221.2, TH233.2, TH245.2, TH257.2, TH269.2, TH281.2, TH29.2, TH293.2, TH305.2, TH41.2, TH5.2, TH53.2, TH65.2, TH77.2, TH89.2
- new net ROW_6: TH102.2, TH114.2, TH126.2, TH138.2, TH150.2, TH162.2, TH174.2, TH18.2, TH186.2, TH198.2, TH210.2, TH222.2, TH234.2, TH246.2, TH258.2, TH270.2, TH282.2, TH294.2, TH30.2, TH306.2, TH42.2, TH54.2, TH6.2, TH66.2, TH78.2, TH90.2
- new net ROW_7: TH103.2, TH115.2, TH127.2, TH139.2, TH151.2, TH163.2, TH175.2, TH187.2, TH19.2, TH199.2, TH211.2, TH223.2, TH235.2, TH247.2, TH259.2, TH271.2, TH283.2, TH295.2, TH307.2, TH31.2, TH43.2, TH55.2, TH67.2, TH7.2, TH79.2, TH91.2
- new net ROW_8: TH104.2, TH116.2, TH128.2, TH140.2, TH152.2, TH164.2, TH176.2, TH188.2, TH20.2, TH200.2, TH212.2, TH224.2, TH236.2, TH248.2, TH260.2, TH272.2, TH284.2, TH296.2, TH308.2, TH32.2, TH44.2, TH56.2, TH68.2, TH8.2, TH80.2, TH92.2
- new net ROW_9: TH105.2, TH117.2, TH129.2, TH141.2, TH153.2, TH165.2, TH177.2, TH189.2, TH201.2, TH21.2, TH213.2, TH225.2, TH237.2, TH249.2, TH261.2, TH273.2, TH285.2, TH297.2, TH309.2, TH33.2, TH45.2, TH57.2, TH69.2, TH81.2, TH9.2, TH93.2
- no-connect marks 45 -> 0
Other:
- note added: "External Header"
- note added: "Thermistor Matrix"
- note removed: "Battery connections"
- note removed: "Circuit Universal Power Input"
- note removed: "Column & Row External connector"
- note removed: "Column Output"
- note removed: "Logic Schematic PCB Version"
- note removed: "Matrix Logic 1"
- note removed: "Matrix Logic 2"
- note removed: "Microcontroller"
- note removed: "Miscellaneous"
- note removed: "More than one USB must never be used on the board at once."
- note removed: "Row Input"
- note removed: "Row input buffers"
- title: Logic Schematic -> Thermistor Schematic

Commit message: Thermistor schematic V1
Parts:
- added H1, H2, H3, H4: Mounting Hole, MountingHole:MountingHole_2.5mm_Pad, symbol Mechanical:MountingHole_Pad
- added TP1, TP10, TP11, TP12, TP13, TP14, TP15, TP16, TP17, TP18, TP19, TP2, TP20, TP21, TP22, TP23, TP24, TP25, TP26, TP27, TP28, TP29, TP3, TP30, TP31, TP32, TP33, TP34, TP35, TP36, TP37, TP38, TP39, TP4, TP5, TP6, TP7, TP8, TP9: TestPoint_Probe, TestPoint:TestPoint_Pad_D1.0mm, symbol Connector:TestPoint_Probe
- J1: footprint (none) -> Connector_PinHeader_2.54mm:PinHeader_2x20_P2.54mm_Vertical
- TH1, TH10, TH100, TH101, TH102, TH103, TH104, TH105, TH106, TH107, TH108, TH109, TH11, TH110, TH111, TH112, TH113, TH114, TH115, TH116, TH117, TH118, TH119, TH12, TH120, TH121, TH122, TH123, TH124, TH125, TH126, TH127, TH128, TH129, TH13, TH130, TH131, TH132, TH133, TH134, TH135, TH136, TH137, TH138, TH139, TH14, TH140, TH141, TH142, TH143, TH144, TH145, TH146, TH147, TH148, TH149, TH15, TH150, TH151, TH152, TH153, TH154, TH155, TH156, TH157, TH158, TH159, TH16, TH160, TH161, TH162, TH163, TH164, TH165, TH166, TH167, TH168, TH169, TH17, TH170, TH171, TH172, TH173, TH174, TH175, TH176, TH177, TH178, TH179, TH18, TH180, TH181, TH182, TH183, TH184, TH185, TH186, TH187, TH188, TH189, TH19, TH190, TH191, TH192, TH193, TH194, TH195, TH196, TH197, TH198, TH199, TH2, TH20, TH200, TH201, TH202, TH203, TH204, TH205, TH206, TH207, TH208, TH209, TH21, TH210, TH211, TH212, TH213, TH214, TH215, TH216, TH217, TH218, TH219, TH22, TH220, TH221, TH222, TH223, TH224, TH225, TH226, TH227, TH228, TH229, TH23, TH230, TH231, TH232, TH233, TH234, TH235, TH236, TH237, TH238, TH239, TH24, TH240, TH241, TH242, TH243, TH244, TH245, TH246, TH247, TH248, TH249, TH25, TH250, TH251, TH252, TH253, TH254, TH255, TH256, TH257, TH258, TH259, TH26, TH260, TH261, TH262, TH263, TH264, TH265, TH266, TH267, TH268, TH269, TH27, TH270, TH271, TH272, TH273, TH274, TH275, TH276, TH277, TH278, TH279, TH28, TH280, TH281, TH282, TH283, TH284, TH285, TH286, TH287, TH288, TH289, TH29, TH290, TH291, TH292, TH293, TH294, TH295, TH296, TH297, TH298, TH299, TH3, TH30, TH300, TH301, TH302, TH303, TH304, TH305, TH306, TH307, TH308, TH309, TH31, TH310, TH311, TH312, TH32, TH33, TH34, TH35, TH36, TH37, TH38, TH39, TH4, TH40, TH41, TH42, TH43, TH44, TH45, TH46, TH47, TH48, TH49, TH5, TH50, TH51, TH52, TH53, TH54, TH55, TH56, TH57, TH58, TH59, TH6, TH60, TH61, TH62, TH63, TH64, TH65, TH66, TH67, TH68, TH69, TH7, TH70, TH71, TH72, TH73, TH74, TH75, TH76, TH77, TH78, TH79, TH8, TH80, TH81, TH82, TH83, TH84, TH85, TH86, TH87, TH88, TH89, TH9, TH90, TH91, TH92, TH93, TH94, TH95, TH96, TH97, TH98, TH99: footprint (none) -> Resistor_THT:R_Axial_DIN0207_L6.3mm_D2.5mm_P7.62mm_Horizontal
Connections:
- net COL_1 is gone; now on net COLUMN_1: TH1.1, TH10.1, TH11.1, TH12.1, TH2.1, TH3.1, TH4.1, TH5.1, TH6.1, TH7.1, TH8.1, TH9.1
- net COL_10 is gone; now on net COLUMN_10: TH109.1, TH110.1, TH111.1, TH112.1, TH113.1, TH114.1, TH115.1, TH116.1, TH117.1, TH118.1, TH119.1, TH120.1
- net COL_11 is gone; now on net COLUMN_11: TH121.1, TH122.1, TH123.1, TH124.1, TH125.1, TH126.1, TH127.1, TH128.1, TH129.1, TH130.1, TH131.1, TH132.1
- net COL_12 is gone; now on net COLUMN_12: TH133.1, TH134.1, TH135.1, TH136.1, TH137.1, TH138.1, TH139.1, TH140.1, TH141.1, TH142.1, TH143.1, TH144.1
- net COL_13 is gone; now on net COLUMN_13: TH145.1, TH146.1, TH147.1, TH148.1, TH149.1, TH150.1, TH151.1, TH152.1, TH153.1, TH154.1, TH155.1, TH156.1
- net COL_14 is gone; now on net COLUMN_14: TH157.1, TH158.1, TH159.1, TH160.1, TH161.1, TH162.1, TH163.1, TH164.1, TH165.1, TH166.1, TH167.1, TH168.1
- net COL_15 is gone; now on net COLUMN_15: TH169.1, TH170.1, TH171.1, TH172.1, TH173.1, TH174.1, TH175.1, TH176.1, TH177.1, TH178.1, TH179.1, TH180.1
- net COL_16 is gone; now on net COLUMN_16: TH181.1, TH182.1, TH183.1, TH184.1, TH185.1, TH186.1, TH187.1, TH188.1, TH189.1, TH190.1, TH191.1, TH192.1
- net COL_17 is gone; now on net COLUMN_17: TH193.1, TH194.1, TH195.1, TH196.1, TH197.1, TH198.1, TH199.1, TH200.1, TH201.1, TH202.1, TH203.1, TH204.1
- net COL_18 is gone; now on net COLUMN_18: TH205.1, TH206.1, TH207.1, TH208.1, TH209.1, TH210.1, TH211.1, TH212.1, TH213.1, TH214.1, TH215.1, TH216.1
- net COL_19 is gone; now on net COLUMN_19: TH217.1, TH218.1, TH219.1, TH220.1, TH221.1, TH222.1, TH223.1, TH224.1, TH225.1, TH226.1, TH227.1, TH228.1
- net COL_2 is gone; now on net COLUMN_2: TH13.1, TH14.1, TH15.1, TH16.1, TH17.1, TH18.1, TH19.1, TH20.1, TH21.1, TH22.1, TH23.1, TH24.1
- net COL_20 is gone; now on net COLUMN_20: TH229.1, TH230.1, TH231.1, TH232.1, TH233.1, TH234.1, TH235.1, TH236.1, TH237.1, TH238.1, TH239.1, TH240.1
- net COL_21 is gone; now on net COLUMN_21: TH241.1, TH242.1, TH243.1, TH244.1, TH245.1, TH246.1, TH247.1, TH248.1, TH249.1, TH250.1, TH251.1, TH252.1
- net COL_22 is gone; now on net COLUMN_22: TH253.1, TH254.1, TH255.1, TH256.1, TH257.1, TH258.1, TH259.1, TH260.1, TH261.1, TH262.1, TH263.1, TH264.1
- net COL_23 is gone; now on net COLUMN_23: TH265.1, TH266.1, TH267.1, TH268.1, TH269.1, TH270.1, TH271.1, TH272.1, TH273.1, TH274.1, TH275.1, TH276.1
- net COL_24 is gone; now on net COLUMN_24: TH277.1, TH278.1, TH279.1, TH280.1, TH281.1, TH282.1, TH283.1, TH284.1, TH285.1, TH286.1, TH287.1, TH288.1
- net COL_25 is gone; now on net COLUMN_25: TH289.1, TH290.1, TH291.1, TH292.1, TH293.1, TH294.1, TH295.1, TH296.1, TH297.1, TH298.1, TH299.1, TH300.1
- net COL_26 is gone; now on net COLUMN_26: TH301.1, TH302.1, TH303.1, TH304.1, TH305.1, TH306.1, TH307.1, TH308.1, TH309.1, TH310.1, TH311.1, TH312.1
- net COL_3 is gone; now on net COLUMN_3: TH25.1, TH26.1, TH27.1, TH28.1, TH29.1, TH30.1, TH31.1, TH32.1, TH33.1, TH34.1, TH35.1, TH36.1
- net COL_4 is gone; now on net COLUMN_4: TH37.1, TH38.1, TH39.1, TH40.1, TH41.1, TH42.1, TH43.1, TH44.1, TH45.1, TH46.1, TH47.1, TH48.1
- net COL_5 is gone; now on net COLUMN_5: TH49.1, TH50.1, TH51.1, TH52.1, TH53.1, TH54.1, TH55.1, TH56.1, TH57.1, TH58.1, TH59.1, TH60.1
- net COL_6 is gone; now on net COLUMN_6: TH61.1, TH62.1, TH63.1, TH64.1, TH65.1, TH66.1, TH67.1, TH68.1, TH69.1, TH70.1, TH71.1, TH72.1
- net COL_7 is gone; now on net COLUMN_7: TH73.1, TH74.1, TH75.1, TH76.1, TH77.1, TH78.1, TH79.1, TH80.1, TH81.1, TH82.1, TH83.1, TH84.1
- net COL_8 is gone; now on net COLUMN_8: TH85.1, TH86.1, TH87.1, TH88.1, TH89.1, TH90.1, TH91.1, TH92.1, TH93.1, TH94.1, TH95.1, TH96.1
- net COL_9 is gone; now on net COLUMN_9: TH100.1, TH101.1, TH102.1, TH103.1, TH104.1, TH105.1, TH106.1, TH107.1, TH108.1, TH97.1, TH98.1, TH99.1
- net ROW_1: now also J1.17 (Pin_17), TP27.1
- net ROW_10: now also J1.35 (Pin_35), TP36.1
- net ROW_11: now also J1.34 (Pin_34), TP37.1
- net ROW_12: now also J1.33 (Pin_33), TP38.1
- net ROW_2: now also J1.18 (Pin_18), TP28.1
- net ROW_3: now also J1.19 (Pin_19), TP29.1
- net ROW_4: now also J1.20 (Pin_20), TP30.1
- net ROW_5: now also J1.40 (Pin_40), TP31.1
- net ROW_6: now also J1.39 (Pin_39), TP32.1
- net ROW_7: now also J1.38 (Pin_38), TP33.1
- net ROW_8: now also J1.37 (Pin_37), TP34.1
- net ROW_9: now also J1.36 (Pin_36), TP35.1
- net COLUMN_16: now reaches J1.1 (Pin_1)
- net COLUMN_16: now also TP16.1
- net COLUMN_24: now reaches J1.10 (Pin_10)
- net COLUMN_24: now also TP24.1
- net COLUMN_25: now reaches J1.11 (Pin_11)
- net COLUMN_25: now also TP25.1
- net COLUMN_26: now reaches J1.12 (Pin_12)
- net COLUMN_26: now also TP26.1
- net COLUMN_20: now reaches J1.13 (Pin_13)
- net COLUMN_20: now also TP20.1
- net COLUMN_19: now reaches J1.14 (Pin_14)
- net COLUMN_19: now also TP19.1
- net COLUMN_18: now reaches J1.15 (Pin_15)
- net COLUMN_18: now also TP18.1
- net COLUMN_17: now reaches J1.16 (Pin_16)
- net COLUMN_17: now also TP17.1
- net COLUMN_15: now reaches J1.2 (Pin_2)
- net COLUMN_15: now also TP15.1
- net COLUMN_12: now reaches J1.21 (Pin_21)
- net COLUMN_12: now also TP12.1
- net COLUMN_11: now reaches J1.22 (Pin_22)
- net COLUMN_11: now also TP11.1
- net COLUMN_10: now reaches J1.23 (Pin_23)
- net COLUMN_10: now also TP10.1
- net COLUMN_9: now reaches J1.24 (Pin_24)
- net COLUMN_9: now also TP9.1
- net COLUMN_5: now reaches J1.25 (Pin_25)
- net COLUMN_5: now also TP5.1
- net COLUMN_6: now reaches J1.26 (Pin_26)
- net COLUMN_6: now also TP6.1
- net COLUMN_7: now reaches J1.27 (Pin_27)
- net COLUMN_7: now also TP7.1
- net COLUMN_8: now reaches J1.28 (Pin_28)
- net COLUMN_8: now also TP8.1
- net COLUMN_22: now reaches J1.29 (Pin_29)
- net COLUMN_22: now also TP22.1
- net COLUMN_14: now reaches J1.3 (Pin_3)
- net COLUMN_14: now also TP14.1
- net COLUMN_21: now reaches J1.30 (Pin_30)
- net COLUMN_21: now also TP21.1
- net GND: now reaches J1.32 (Pin_32)
- net GND: now also H1.1, H2.1, H3.1, H4.1, TP39.1
- net COLUMN_13: now reaches J1.4 (Pin_4)
- net COLUMN_13: now also TP13.1
- net COLUMN_1: now reaches J1.5 (Pin_5)
- net COLUMN_1: now also TP1.1
- net COLUMN_2: now reaches J1.6 (Pin_6)
- net COLUMN_2: now also TP2.1
- net COLUMN_3: now reaches J1.7 (Pin_7)
- net COLUMN_3: now also TP3.1
- net COLUMN_4: now reaches J1.8 (Pin_8)
- net COLUMN_4: now also TP4.1
- net COLUMN_23: now reaches J1.9 (Pin_9)
- net COLUMN_23: now also TP23.1
- no-connect marks 0 -> 1
Other:
- note added: "Miscellaneous"
- moved on the sheet: J1, TH1, TH10, TH100, TH101, TH102, TH103, TH104, TH105, TH106, TH107, TH108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

Commit message: Work on V2 thermistor PCB
Parts:
- removed J1: Header, Connector_PinHeader_2.54mm:PinHeader_2x20_P2.54mm_Vertical, symbol Connector_Generic:Conn_02x20_Top_Bottom
- removed TH1, TH10, TH100, TH101, TH102, TH103, TH104, TH105, TH106, TH107, TH108, TH109, TH11, TH110, TH111, TH112, TH113, TH114, TH115, TH116, TH117, TH118, TH119, TH12, TH120, TH121, TH122, TH123, TH124, TH125, TH126, TH127, TH128, TH129, TH13, TH130, TH131, TH132, TH133, TH134, TH135, TH136, TH137, TH138, TH139, TH14, TH140, TH141, TH142, TH143, TH144, TH145, TH146, TH147, TH148, TH149, TH15, TH150, TH151, TH152, TH153, TH154, TH155, TH156, TH157, TH158, TH159, TH16, TH160, TH161, TH162, TH163, TH164, TH165, TH166, TH167, TH168, TH169, TH17, TH170, TH171, TH172, TH173, TH174, TH175, TH176, TH177, TH178, TH179, TH18, TH180, TH181, TH182, TH183, TH184, TH185, TH186, TH187, TH188, TH189, TH19, TH190, TH191, TH192, TH193, TH194, TH195, TH196, TH197, TH198, TH199, TH2, TH20, TH200, TH201, TH202, TH203, TH204, TH205, TH206, TH207, TH208, TH209, TH21, TH210, TH211, TH212, TH213, TH214, TH215, TH216, TH217, TH218, TH219, TH22, TH220, TH221, TH222, TH223, TH224, TH225, TH226, TH227, TH228, TH229, TH23, TH230, TH231, TH232, TH233, TH234, TH235, TH236, TH237, TH238, TH239, TH24, TH240, TH241, TH242, TH243, TH244, TH245, TH246, TH247, TH248, TH249, TH25, TH250, TH251, TH252, TH253, TH254, TH255, TH256, TH257, TH258, TH259, TH26, TH260, TH261, TH262, TH263, TH264, TH265, TH266, TH267, TH268, TH269, TH27, TH270, TH271, TH272, TH273, TH274, TH275, TH276, TH277, TH278, TH279, TH28, TH280, TH281, TH282, TH283, TH284, TH285, TH286, TH287, TH288, TH289, TH29, TH290, TH291, TH292, TH293, TH294, TH295, TH296, TH297, TH298, TH299, TH3, TH30, TH300, TH301, TH302, TH303, TH304, TH305, TH306, TH307, TH308, TH309, TH31, TH310, TH311, TH312, TH32, TH33, TH34, TH35, TH36, TH37, TH38, TH39, TH4, TH40, TH41, TH42, TH43, TH44, TH45, TH46, TH47, TH48, TH49, TH5, TH50, TH51, TH52, TH53, TH54, TH55, TH56, TH57, TH58, TH59, TH6, TH60, TH61, TH62, TH63, TH64, TH65, TH66, TH67, TH68, TH69, TH7, TH70, TH71, TH72, TH73, TH74, TH75, TH76, TH77, TH78, TH79, TH8, TH80, TH81, TH82, TH83, TH84, TH85, TH86, TH87, TH88, TH89, TH9, TH90, TH91, TH92, TH93, TH94, TH95, TH96, TH97, TH98, TH99: 10k, Resistor_THT:R_Axial_DIN0207_L6.3mm_D2.5mm_P7.62mm_Horizontal, symbol Device:Thermistor_NTC_US
- removed TP13, TP14, TP15, TP16, TP17, TP18, TP19, TP20, TP21, TP22, TP23, TP24, TP25, TP26, TP27, TP28, TP29, TP30, TP31, TP32, TP33, TP34, TP35, TP36, TP37, TP38: TestPoint_Probe, TestPoint:TestPoint_Pad_D1.0mm, symbol Connector:TestPoint_Probe
- added J1: Header, Connector_PinHeader_2.54mm:PinHeader_2x20_P2.54mm_Vertical, symbol Connector_Generic:Conn_02x20_Odd_Even
- renumbered TP39 to TP13
Connections:
- net COLUMN_1: now also J1.10 (Pin_10); no longer TP1.1
- net COLUMN_10: now also J1.5 (Pin_5); no longer TP10.1
- net COLUMN_11: now also J1.3 (Pin_3); no longer TP11.1
- net COLUMN_12: now also J1.1 (Pin_1); no longer TP12.1
- net COLUMN_13: now also J1.8 (Pin_8)
- net COLUMN_14: now also J1.6 (Pin_6)
- net COLUMN_15: now also J1.4 (Pin_4)
- net COLUMN_16: now also J1.2 (Pin_2)
- net COLUMN_17: now also J1.32 (Pin_32)
- net COLUMN_18: now also J1.30 (Pin_30)
- net COLUMN_19: now also J1.28 (Pin_28)
- net COLUMN_2: now also J1.12 (Pin_12); no longer TP2.1
- net COLUMN_20: now also J1.26 (Pin_26)
- net COLUMN_21: now also J1.19 (Pin_19)
- net COLUMN_22: now also J1.17 (Pin_17)
- net COLUMN_23: now also J1.18 (Pin_18)
- net COLUMN_24: now also J1.20 (Pin_20)
- net COLUMN_25: now also J1.22 (Pin_22)
- net COLUMN_26: now also J1.24 (Pin_24)
- net COLUMN_3: now also J1.14 (Pin_14); no longer TP3.1
- net COLUMN_4: now also J1.16 (Pin_16); no longer TP4.1
- net COLUMN_5: now also J1.9 (Pin_9); no longer TP5.1
- net COLUMN_6: now also J1.11 (Pin_11); no longer TP6.1
- net COLUMN_7: now also J1.13 (Pin_13); no longer TP7.1
- net COLUMN_8: now also J1.15 (Pin_15); no longer TP8.1
- net COLUMN_9: now also J1.7 (Pin_7); no longer TP9.1
- net GND: now also J1.23 (Pin_23)
- net ROW_1: now also TP1.1, J1.34 (Pin_34)
- net ROW_10: now also TP10.1, J1.29 (Pin_29)
- net ROW_11: now also TP11.1, J1.27 (Pin_27)
- net ROW_12: now also TP12.1, J1.25 (Pin_25)
- net ROW_2: now also TP2.1, J1.36 (Pin_36)
- net ROW_3: now also TP3.1, J1.38 (Pin_38)
- net ROW_4: now also TP4.1, J1.40 (Pin_40)
- net ROW_5: now also TP5.1, J1.39 (Pin_39)
- net ROW_6: now also TP6.1, J1.37 (Pin_37)
- net ROW_7: now also TP7.1, J1.35 (Pin_35)
- net ROW_8: now also TP8.1, J1.33 (Pin_33)
- net ROW_9: now also TP9.1, J1.31 (Pin_31)
Other:
- added sheet Thermistor Column Cell (thermistor_c_cell.kicad_sch)
- added sheet Thermistor Column Cell1 (thermistor_c_cell.kicad_sch)
- added sheet Thermistor Column Cell10 (thermistor_c_cell.kicad_sch)
- added sheet Thermistor Column Cell11 (thermistor_c_cell.kicad_sch)
- added sheet Thermistor Column Cell12 (thermistor_c_cell.kicad_sch)
- added sheet Thermistor Column Cell13 (thermistor_c_cell.kicad_sch)
- added sheet Thermistor Column Cell14 (thermistor_c_cell.kicad_sch)
- added sheet Thermistor Column Cell15 (thermistor_c_cell.kicad_sch)
- added sheet Thermistor Column Cell16 (thermistor_c_cell.kicad_sch)
- added sheet Thermistor Column Cell17 (thermistor_c_cell.kicad_sch)
- added sheet Thermistor Column Cell18 (thermistor_c_cell.kicad_sch)
- added sheet Thermistor Column Cell19 (thermistor_c_cell.kicad_sch)
- added sheet Thermistor Column Cell2 (thermistor_c_cell.kicad_sch)
- added sheet Thermistor Column Cell20 (thermistor_c_cell.kicad_sch)
- added sheet Thermistor Column Cell21 (thermistor_c_cell.kicad_sch)
- added sheet Thermistor Column Cell22 (thermistor_c_cell.kicad_sch)
- added sheet Thermistor Column Cell23 (thermistor_c_cell.kicad_sch)
- added sheet Thermistor Column Cell24 (thermistor_c_cell.kicad_sch)
- added sheet Thermistor Column Cell25 (thermistor_c_cell.kicad_sch)
- added sheet Thermistor Column Cell3 (thermistor_c_cell.kicad_sch)
- added sheet Thermistor Column Cell4 (thermistor_c_cell.kicad_sch)
- added sheet Thermistor Column Cell5 (thermistor_c_cell.kicad_sch)
- added sheet Thermistor Column Cell6 (thermistor_c_cell.kicad_sch)
- added sheet Thermistor Column Cell7 (thermistor_c_cell.kicad_sch)
- added sheet Thermistor Column Cell8 (thermistor_c_cell.kicad_sch)
- added sheet Thermistor Column Cell9 (thermistor_c_cell.kicad_sch)
- moved on the sheet: H1, H2, H3, H4, TP13
