File: Finalized Thermistor Schematic/inventeam_thermistor_schematic/inventeam_thermistor_schematic.kicad_pcb (KiCad board)
At the start: 2 copper layers, 356 parts, among them J1 Header

Commit message: Work on V2 thermistor PCB
Parts:
- TH1, TH10, TH100, TH101, TH102, TH103, TH104, TH105, TH106, TH107, TH108, TH109, TH11, TH110, TH111, TH112, TH113, TH114, TH115, TH116, TH117, TH118, TH119, TH12, TH120, TH121, TH122, TH123, TH124, TH125, TH126, TH127, TH128, TH129, TH13, TH130, TH131, TH132, TH133, TH134, TH135, TH136, TH137, TH138, TH139, TH14, TH140, TH141, TH142, TH143, TH144, TH145, TH146, TH147, TH148, TH149, TH15, TH150, TH151, TH152, TH153, TH154, TH155, TH156, TH157, TH158, TH159, TH16, TH160, TH161, TH162, TH163, TH164, TH165, TH166, TH167, TH168, TH169, TH17, TH170, TH171, TH172, TH173, TH174, TH175, TH176, TH177, TH178, TH179, TH18, TH180, TH181, TH182, TH183, TH184, TH185, TH186, TH187, TH188, TH189, TH19, TH190, TH191, TH192, TH193, TH194, TH195, TH196, TH197, TH198, TH199, TH2, TH20, TH200, TH201, TH202, TH203, TH204, TH205, TH206, TH207, TH208, TH209, TH21, TH210, TH211, TH212, TH213, TH214, TH215, TH216, TH217, TH218, TH219, TH22, TH220, TH221, TH222, TH223, TH224, TH225, TH226, TH227, TH228, TH229, TH23, TH230, TH231, TH232, TH233, TH234, TH235, TH236, TH237, TH238, TH239, TH24, TH240, TH241, TH242, TH243, TH244, TH245, TH246, TH247, TH248, TH249, TH25, TH250, TH251, TH252, TH253, TH254, TH255, TH256, TH257, TH258, TH259, TH26, TH260, TH261, TH262, TH263, TH264, TH265, TH266, TH267, TH268, TH269, TH27, TH270, TH271, TH272, TH273, TH274, TH275, TH276, TH277, TH278, TH279, TH28, TH280, TH281, TH282, TH283, TH284, TH285, TH286, TH287, TH288, TH289, TH29, TH290, TH291, TH292, TH293, TH294, TH295, TH296, TH297, TH298, TH299, TH3, TH30, TH300, TH301, TH302, TH303, TH304, TH305, TH306, TH307, TH308, TH309, TH31, TH310, TH311, TH312, TH32, TH33, TH34, TH35, TH36, TH37, TH38, TH39, TH4, TH40, TH41, TH42, TH43, TH44, TH45, TH46, TH47, TH48, TH49, TH5, TH50, TH51, TH52, TH53, TH54, TH55, TH56, TH57, TH58, TH59, TH6, TH60, TH61, TH62, TH63, TH64, TH65, TH66, TH67, TH68, TH69, TH7, TH70, TH71, TH72, TH73, TH74, TH75, TH76, TH77, TH78, TH79, TH8, TH80, TH81, TH82, TH83, TH84, TH85, TH86, TH87, TH88, TH89, TH9, TH90, TH91, TH92, TH93, TH94, TH95, TH96, TH97, TH98, TH99: footprint Resistor_THT:R_Axial_DIN0207_L6.3mm_D2.5mm_P7.62mm_Horizontal -> Resistor_THT:R_Axial_DIN0207_L6.3mm_D2.5mm_P2.54mm_Vertical
- moved H4 386.6 mm to (304.9, 160.7)
- moved H2 348.2 mm to (304.9, 30.7)
- moved TP39 312.5 mm to (295.7, 45.6)
- moved TP38 303.7 mm to (286.7, 45.6)
- moved TP37 294.9 mm to (277.7, 45.6)
- moved TP36 286.1 mm to (268.7, 45.6)
- moved TP35 277.4 mm to (259.7, 45.6)
- moved TP34 268.7 mm to (250.7, 45.6)
- moved TP33 260.1 mm to (241.7, 45.6)
- moved TP32 248.8 mm to (232.7, 45.6)
- moved TP31 239.7 mm to (223.7, 45.6)
- moved TP30 230.6 mm to (214.7, 45.6)
- moved TP29 221.6 mm to (205.7, 45.6)
- moved TP28 212.7 mm to (196.7, 45.6)
- moved TP27 203.8 mm to (187.7, 45.6)
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Connections:
- J1 pad 1: COLUMN_16 -> COLUMN_12
- J1 pad 10: COLUMN_24 -> COLUMN_1
- J1 pad 11: COLUMN_25 -> COLUMN_6
- J1 pad 12: COLUMN_26 -> COLUMN_2
- J1 pad 13: COLUMN_20 -> COLUMN_7
- J1 pad 14: COLUMN_19 -> COLUMN_3
- J1 pad 15: COLUMN_18 -> COLUMN_8
- J1 pad 16: COLUMN_17 -> COLUMN_4
- J1 pad 17: ROW_1 -> COLUMN_22
- J1 pad 18: ROW_2 -> COLUMN_23
- J1 pad 19: ROW_3 -> COLUMN_21
- J1 pad 2: COLUMN_15 -> COLUMN_16
- J1 pad 20: ROW_4 -> COLUMN_24
- J1 pad 21: COLUMN_12 -> unconnected-(J1-Pin_21-Pad21)
- J1 pad 22: COLUMN_11 -> COLUMN_25
- J1 pad 23: COLUMN_10 -> GND
- J1 pad 24: COLUMN_9 -> COLUMN_26
- J1 pad 25: COLUMN_5 -> ROW_12
- J1 pad 26: COLUMN_6 -> COLUMN_20
- J1 pad 27: COLUMN_7 -> ROW_11
- J1 pad 28: COLUMN_8 -> COLUMN_19
- J1 pad 29: COLUMN_22 -> ROW_10
- J1 pad 3: COLUMN_14 -> COLUMN_11
- J1 pad 30: COLUMN_21 -> COLUMN_18
- J1 pad 31: unconnected-(J1-Pin_31-Pad31) -> ROW_9
- J1 pad 32: GND -> COLUMN_17
- J1 pad 33: ROW_12 -> ROW_8
- J1 pad 34: ROW_11 -> ROW_1
- J1 pad 35: ROW_10 -> ROW_7
- J1 pad 36: ROW_9 -> ROW_2
- J1 pad 37: ROW_8 -> ROW_6
- J1 pad 38: ROW_7 -> ROW_3
- J1 pad 39: ROW_6 -> ROW_5
- J1 pad 4: COLUMN_13 -> COLUMN_15
- J1 pad 40: ROW_5 -> ROW_4
- J1 pad 5: COLUMN_1 -> COLUMN_10
- J1 pad 6: COLUMN_2 -> COLUMN_14
- J1 pad 7: COLUMN_3 -> COLUMN_9
- J1 pad 8: COLUMN_4 -> COLUMN_13
- J1 pad 9: COLUMN_23 -> COLUMN_5
- TP1 pad 1: COLUMN_1 -> ROW_1
- TP10 pad 1: COLUMN_10 -> ROW_10
- TP11 pad 1: COLUMN_11 -> ROW_11
- TP12 pad 1: COLUMN_12 -> ROW_12
- TP13 pad 1: COLUMN_13 -> GND
- TP14 pad 1: COLUMN_14 -> COLUMN_1
- TP15 pad 1: COLUMN_15 -> COLUMN_2
- TP16 pad 1: COLUMN_16 -> COLUMN_3
- TP17 pad 1: COLUMN_17 -> COLUMN_4
- TP18 pad 1: COLUMN_18 -> COLUMN_5
- TP19 pad 1: COLUMN_19 -> COLUMN_6
- TP2 pad 1: COLUMN_2 -> ROW_2
- TP20 pad 1: COLUMN_20 -> COLUMN_7
- TP21 pad 1: COLUMN_21 -> COLUMN_8
- TP22 pad 1: COLUMN_22 -> COLUMN_9
- TP23 pad 1: COLUMN_23 -> COLUMN_10
- TP24 pad 1: COLUMN_24 -> COLUMN_11
- TP25 pad 1: COLUMN_25 -> COLUMN_12
- TP26 pad 1: COLUMN_26 -> COLUMN_13
- TP27 pad 1: ROW_1 -> COLUMN_14
- TP28 pad 1: ROW_2 -> COLUMN_15
- TP29 pad 1: ROW_3 -> COLUMN_16
- TP3 pad 1: COLUMN_3 -> ROW_3
- TP30 pad 1: ROW_4 -> COLUMN_17
- TP31 pad 1: ROW_5 -> COLUMN_18
- TP32 pad 1: ROW_6 -> COLUMN_19
- TP33 pad 1: ROW_7 -> COLUMN_20
- TP34 pad 1: ROW_8 -> COLUMN_21
- TP35 pad 1: ROW_9 -> COLUMN_22
- TP36 pad 1: ROW_10 -> COLUMN_23
- TP37 pad 1: ROW_11 -> COLUMN_24
- TP38 pad 1: ROW_12 -> COLUMN_25
- TP39 pad 1: GND -> COLUMN_26
- TP4 pad 1: COLUMN_4 -> ROW_4
- TP5 pad 1: COLUMN_5 -> ROW_5
- TP6 pad 1: COLUMN_6 -> ROW_6
- TP7 pad 1: COLUMN_7 -> ROW_7
- TP8 pad 1: COLUMN_8 -> ROW_8
- TP9 pad 1: COLUMN_9 -> ROW_9
Routing:
- net COLUMN_21: track 0.00 -> 464.8 mm, vias 0 -> 1
- net COLUMN_22: track 0.00 -> 464.8 mm, vias 0 -> 1
- net ROW_12: track 0.00 -> 369.3 mm, vias 0 -> 1
- net ROW_11: track 0.00 -> 366.2 mm, vias 0 -> 1
- net ROW_10: track 0.00 -> 362.1 mm, vias 0 -> 1
- net ROW_6: track 0.00 -> 360.3 mm, vias 0 -> 1
- net ROW_8: track 0.00 -> 360.1 mm, vias 0 -> 1
- net ROW_7: track 0.00 -> 359.9 mm, vias 0 -> 1
- net ROW_1: track 0.00 -> 359.3 mm, vias 0 -> 1
- net ROW_9: track 0.00 -> 358.0 mm, vias 0 -> 1
- net COLUMN_16: track 0.00 -> 357.7 mm, vias 0 -> 1
- net ROW_2: track 0.00 -> 353.0 mm, vias 0 -> 1
- net ROW_5: track 0.00 -> 352.4 mm, vias 0 -> 1
- net COLUMN_15: track 0.00 -> 347.9 mm, vias 0 -> 1
- net ROW_3: track 0.00 -> 346.1 mm, vias 0 -> 1
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Other:
- board text added: "C1"
- board text added: "C10"
- board text added: "C11"
- board text added: "C12"
- board text added: "C13"
- board text added: "C14"
- board text added: "C15"
- board text added: "C16"
- board text added: "C17"
- board text added: "C18"
- board text added: "C19"
- board text added: "C2"
- board text added: "C20"
- board text added: "C21"
- board text added: "C22"
- board text added: "C23"
- board text added: "C24"
- board text added: "C25"
- board text added: "C26"
- board text added: "C3"
- board text added: "C4"
- board text added: "C5"
- board text added: "C6"
- board text added: "C7"
- board text added: "C8"
- board text added: "C9"
- board text added: "GND"
- board text added: "R1"
- board text added: "R10"
- board text added: "R11"
- board text added: "R12"
- board text added: "R2"
- board text added: "R3"
- board text added: "R4"
- board text added: "R5"
- board text added: "R6"
- board text added: "R7"
- board text added: "R8"
- board text added: "R9"

Commit message: Finishead header connections
Parts:
- moved H3 4.24 mm to (27.9, 157.7)
- moved H4 4.24 mm to (301.9, 157.7)
- moved H1 4.24 mm to (27.9, 33.7)
- moved H2 4.24 mm to (301.9, 33.7)
Routing:
- net COLUMN_26: track 165.8 -> 470.3 mm, vias 0 -> 1
- net COLUMN_25: track 165.8 -> 461.4 mm, vias 0 -> 1
- net COLUMN_24: track 165.8 -> 452.8 mm, vias 0 -> 1
- net COLUMN_23: track 165.8 -> 444.4 mm, vias 0 -> 1
- net COLUMN_19: track 165.8 -> 412.9 mm, vias 0 -> 1
- net COLUMN_20: track 165.8 -> 408.8 mm, vias 0 -> 1
- net COLUMN_18: track 165.8 -> 385.5 mm, vias 0 -> 1
- net COLUMN_17: track 165.8 -> 378.9 mm, vias 0 -> 1
- net COLUMN_4: track 165.8 -> 262.6 mm, vias 0 -> 1
- net COLUMN_3: track 165.8 -> 249.0 mm, vias 0 -> 1
- net COLUMN_8: track 338.6 -> 333.1 mm
- net COLUMN_7: track 323.2 -> 317.8 mm
- net COLUMN_22: track 464.8 -> 459.4 mm
- net COLUMN_6: track 307.6 -> 302.3 mm
- net COLUMN_9: track 319.8 -> 314.6 mm
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Other:
- board outline added: 280 x 130 mm

Commit message: Thermistor finalized V2
Parts:
- added G***: LOGO, LOGO, F.Cu at (39.7, 44.6)
- added kibuzzard-69C4C75F: G***, kibuzzard-69C4C75F, F.Cu at (67.0, 34.6)
- added kibuzzard-69C4C7E1: G***, kibuzzard-69C4C7E1, F.Cu at (103.0, 33.6)
- added kibuzzard-69C4C905: G***, kibuzzard-69C4C905, F.Cu at (291.8, 159.0)
- moved H1 1.58 mm to (26.4, 34.2)
- moved H2 1.58 mm to (303.4, 34.2)
- moved H3 1.58 mm to (26.4, 157.2)
- moved H4 1.58 mm to (303.4, 157.2)
Routing:
- net COLUMN_18: track 385.5 -> 384.0 mm
- added copper zone on B.Cu, net GND
- added copper zone on F.Cu, net GND
Other:
- board size 280 x 130 mm -> 287 x 133 mm
