File: Finalized Pressure Schematic/Column Schematic/pressure_column_schematic/column_cell.kicad_sch (KiCad schematic)
At the start: 0 parts

Commit message: Work on V1
Parts:
- added TP1, TP10, TP11, TP12, TP2, TP3, TP4, TP5, TP6, TP7, TP8, TP9: TestPoint, symbol Connector:TestPoint
Connections:
- new net COL_OUT: TP1.1, TP10.1, TP11.1, TP12.1, TP2.1, TP3.1, TP4.1, TP5.1, TP6.1, TP7.1, TP8.1, TP9.1
Other:
- note added: "LionStride"
