File: Finalized Pressure Schematic/Row Schematic/pressure_row_schematic/pressure_row_schematic.kicad_sch (KiCad schematic)
At the start: 0 parts

Commit message: initialized hierarchal sheets
Other:
- added sheet Row Cell (row_cell.kicad_sch)
- note added: "LionStride"

Commit message: Worked on V1
Parts:
- added J1: Conn_01x12, symbol Connector_Generic:Conn_01x12
Connections:
- new net ROW_1: J1.1 (Pin_1)
- new net ROW_10: J1.10 (Pin_10)
- new net ROW_11: J1.11 (Pin_11)
- new net ROW_12: J1.12 (Pin_12)
- new net ROW_2: J1.2 (Pin_2)
- new net ROW_3: J1.3 (Pin_3)
- new net ROW_4: J1.4 (Pin_4)
- new net ROW_5: J1.5 (Pin_5)
- new net ROW_6: J1.6 (Pin_6)
- new net ROW_7: J1.7 (Pin_7)
- new net ROW_8: J1.8 (Pin_8)
- new net ROW_9: J1.9 (Pin_9)
Other:
- added sheet Row Cell1 (row_cell.kicad_sch)
- added sheet Row Cell10 (row_cell.kicad_sch)
- added sheet Row Cell11 (row_cell.kicad_sch)
- added sheet Row Cell2 (row_cell.kicad_sch)
- added sheet Row Cell3 (row_cell.kicad_sch)
- added sheet Row Cell4 (row_cell.kicad_sch)
- added sheet Row Cell5 (row_cell.kicad_sch)
- added sheet Row Cell6 (row_cell.kicad_sch)
- added sheet Row Cell7 (row_cell.kicad_sch)
- added sheet Row Cell8 (row_cell.kicad_sch)
- added sheet Row Cell9 (row_cell.kicad_sch)
- sheet Row Cell ports: added ROW_OUT; removed none
- note added: "Output"
- note added: "Rows"

Commit message: Added missing revision date and title
Other:
- title: (none) -> Pressure Row Schematic
Changed lines of the file:
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@@
 	(generator_version "9.0")
 	(paper "User" 152.4 254)
+	(title_block
+		(title "Pressure Row Schematic")
+		(date "2026-04-11")
+	)
 	(rectangle
 		(start 13.97 13.97)
