File: Finalized Schematics/Finalized Pressure Schematic/inventeam_pressure_schematic/pressure_matrix.kicad_sch (KiCad schematic)
At the start: 26 parts, among them U1 ColumnPad, U10 ColumnPad, U11 ColumnPad, U12 ColumnPad, U13 ColumnPad, U14 ColumnPad, U15 ColumnPad, U16 ColumnPad, U17 ColumnPad, U18 ColumnPad, U19 ColumnPad, U2 ColumnPad, U20 ColumnPad, U21 ColumnPad, U22 ColumnPad, U23 ColumnPad, U24 ColumnPad, U25 ColumnPad, U26 ColumnPad, U3 ColumnPad, U4 ColumnPad, U5 ColumnPad, U6 ColumnPad, U7 ColumnPad, U8 ColumnPad, U9 ColumnPad

Commit message: Pressure V2.1
Parts:
- removed U1, U10, U11, U12, U13, U14, U15, U16, U17, U18, U19, U2, U20, U21, U22, U23, U24, U25, U26, U3, U4, U5, U6, U7, U8, U9: ColumnPad, symbol pressure_pads:Column_pad
Connections:
- no-connect marks 0 -> 38
Other:
- note added: "Pressure Matrix"
- title: Column Matrix -> Row Matrix
