File: Finalized Schematics/Finalized Pressure Schematic/inventeam_pressure_schematic/inventeam_pressure_schematic.kicad_pcb (KiCad board)
At the start: 4 copper layers, 43 parts, among them J1 Conn_02x20_Odd_Even

Commit message: Pressure V2.2
Parts:
- added G***: LOGO, LOGO, F.Cu at (61.5, 192.5)
- added TP39: TestPoint_Probe, TestPoint:TestPoint_Pad_D2.5mm, F.Cu at (71.5, 74.4)
- added kibuzzard-69F7F9B9: G***, kibuzzard-69F7F9B9, F.Cu at (107.4, 205.6)
- added kibuzzard-69F7FA32: G***, kibuzzard-69F7FA32, F.Cu at (151.9, 206.1)
- added kibuzzard-69F7FCC3: G***, kibuzzard-69F7FCC3, F.Cu at (100.4, 57.0)
- added kibuzzard-69F7FCD4: G***, kibuzzard-69F7FCD4, F.Cu at (82.0, 68.0)
- added kibuzzard-69F7FD79: G***, kibuzzard-69F7FD79, F.Cu at (357.7, 210.1)
- added kibuzzard-69F8111F: G***, kibuzzard-69F8111F, F.Cu at (71.5, 68.0)
- added kibuzzard-69F81189: G***, kibuzzard-69F81189, F.Cu at (182.0, 205.0)
- moved H3 441.1 mm to (46.7, 209.7)
- moved H1 437.5 mm to (46.7, 55.7)
- moved H4 128.3 mm to (375.7, 209.7)
- moved H2 123.4 mm to (375.7, 55.7)
Routing:
- net COL_22: track 0.00 -> 344.3 mm, vias 0 -> 1
- net COL_26: track 0.00 -> 342.1 mm, vias 0 -> 1
- net COL_25: track 0.00 -> 330.0 mm, vias 0 -> 1
- net COL_21: track 0.00 -> 325.9 mm, vias 0 -> 1
- net COL_24: track 0.00 -> 317.9 mm, vias 0 -> 1
- net COL_23: track 0.00 -> 305.9 mm, vias 0 -> 1
- net COL_12: track 0.00 -> 284.6 mm, vias 0 -> 1
- net COL_20: track 0.00 -> 282.8 mm, vias 0 -> 1
- net COL_19: track 0.00 -> 270.5 mm, vias 0 -> 1
- net COL_11: track 0.00 -> 265.6 mm, vias 0 -> 1
- net COL_18: track 0.00 -> 258.2 mm, vias 0 -> 1
- net COL_10: track 0.00 -> 247.3 mm, vias 0 -> 1
- net COL_17: track 0.00 -> 246.0 mm, vias 0 -> 1
- net COL_16: track 0.00 -> 244.1 mm, vias 0 -> 1
- net COL_15: track 0.00 -> 231.9 mm, vias 0 -> 1
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- added copper zone on B.Cu, net GND
- added copper zone on F.Cu, net GND
- added copper zone on In1.Cu, net GND
Other:
- board outline added: 335 x 160 mm
